Commit message: updating URDF for eyes including inertia matrices and orientation

File: romeo_description/urdf/romeo_generated_urdf/romeo_eyes.xacro (robot description, xacro)
@@ -14,6 +14,6 @@
 		<inertial>
 			<mass value="0.01"/>
-			<inertia ixx="0" ixy="0" ixz="0" iyy="0" iyz="0" izz="0"/>
-			<origin rpy="0 0 0" xyz="0 0 0"/>
+			<inertia ixx="1e-09" ixy="0" ixz="0" iyy="1e-09" iyz="0" izz="1e-09" />
+			<origin rpy="0 -0 1.5708" xyz="0 0 0"/>
 		</inertial>
 	</link>
@@ -28,6 +28,6 @@
 		<inertial>
 			<mass value="0.01"/>
-			<inertia ixx="0" ixy="0" ixz="0" iyy="0" iyz="0" izz="0"/>
-			<origin rpy="0 0 0" xyz="0 0 0"/>
+			<inertia ixx="1e-09" ixy="0" ixz="0" iyy="1e-09" iyz="0" izz="1e-09" />
+			<origin rpy="1.5708 -0 -3.14159" xyz="0 0 0"/>
 		</inertial>
 		<xacro:insert_visu_LEye/>
@@ -43,6 +43,6 @@
 		<inertial>
 			<mass value="0.01"/>
-			<inertia ixx="0" ixy="0" ixz="0" iyy="0" iyz="0" izz="0"/>
-			<origin rpy="0 0 0" xyz="0 0 0"/>
+			<inertia ixx="1e-09" ixy="0" ixz="0" iyy="1e-09" iyz="0" izz="1e-09" />
+			<origin rpy="0 -0 1.5708" xyz="0 0 0"/>
 		</inertial>
 	</link>
@@ -57,6 +57,6 @@
 		<inertial>
 			<mass value="0.01"/>
-			<inertia ixx="0" ixy="0" ixz="0" iyy="0" iyz="0" izz="0"/>
-			<origin rpy="0 0 0" xyz="0 0 0"/>
+			<inertia ixx="1e-09" ixy="0" ixz="0" iyy="1e-09" iyz="0" izz="1e-09" />
+			<origin rpy="1.5708 -0 -3.14159" xyz="0 0 0"/>
 		</inertial>
 		<xacro:insert_visu_REye/>

Commit message: adding back the inertia matrices for eyes

File: romeo_description/urdf/romeo_generated_urdf/romeo_eyes.xacro (robot description, xacro)
@@ -14,5 +14,5 @@
 		<inertial>
 			<mass value="0.01"/>
-			<inertia ixx="0" ixy="0" ixz="0" iyy="0" iyz="0" izz="0"/>
+			<inertia ixx="1e-09" ixy="0" ixz="0" iyy="1e-09" iyz="0" izz="1e-09" />
 			<origin rpy="0 0 1.5708" xyz="0 0 0"/>
 		</inertial>
@@ -28,5 +28,5 @@
 		<inertial>
 			<mass value="0.01"/>
-			<inertia ixx="0" ixy="0" ixz="0" iyy="0" iyz="0" izz="0"/>
+			<inertia ixx="1e-09" ixy="0" ixz="0" iyy="1e-09" iyz="0" izz="1e-09" />
 			<origin rpy="1.5708 0 -3.14159" xyz="0 0 0"/>
 		</inertial>
@@ -43,5 +43,5 @@
 		<inertial>
 			<mass value="0.01"/>
-			<inertia ixx="0" ixy="0" ixz="0" iyy="0" iyz="0" izz="0"/>
+			<inertia ixx="1e-09" ixy="0" ixz="0" iyy="1e-09" iyz="0" izz="1e-09" />
 			<origin rpy="0 0 1.5708" xyz="0 0 0"/>
 		</inertial>
@@ -57,5 +57,5 @@
 		<inertial>
 			<mass value="0.01"/>
-			<inertia ixx="0" ixy="0" ixz="0" iyy="0" iyz="0" izz="0"/>
+			<inertia ixx="1e-09" ixy="0" ixz="0" iyy="1e-09" iyz="0" izz="1e-09" />
 			<origin rpy="1.5708 0 -3.14159" xyz="0 0 0"/>
 		</inertial>
