Commit message: Updating CameraDepth_frame with an additional optical frame

File: romeo_description/urdf/romeo_generated_urdf/romeo_cap.xacro (robot description, xacro)
@@ -9,8 +9,14 @@
 <robot xmlns:xacro="http://www.ros.org/wiki/xacro">
     <link name="CameraDepth_frame"/>
-    <joint name="CameraDepth_joint" type="fixed">
-        <parent link="HeadRoll_link"/>
-        <child link="CameraDepth_frame"/>
-        <origin rpy="2.0043951 0 1.57079632679" xyz="0.1403 -0.04708 0.14655"/>
+	<joint name="CameraDepth_joint" type="fixed">
+		<parent link="HeadRoll_link"/>
+		<child link="CameraDepth_frame"/>
+		<origin rpy="0 0 0" xyz="0.1403 -0.04708 0.14655"/>
+    </joint>
+    <link name="CameraDepth_optical_frame"/>
+	<joint name="CameraDepth_optical_frame_fixedjoint" type="fixed">
+		<parent link="CameraDepth_frame"/>
+		<child link="CameraDepth_optical_frame"/>
+		<origin rpy="2.0043951 0 1.57079632679" xyz="0 0 0"/>
     </joint>
     <link name="Cap">
