Commit message: added romeo cap with xtion to meshes and urdf

File: romeo_description/urdf/romeo_generated_urdf/romeo.urdf (robot description, URDF)
Before this commit: robot romeoH37, 90 links, 89 joints
Links:
- added link CameraDepth_frame
- added link Cap, mass 0.29923; visual mesh filename=package://romeo_description/meshes/Cap.dae scale=1 1 1
Joints:
- added joint CameraDepth_joint: type fixed, parent HeadRoll_link, child CameraDepth_frame, origin xyz=0.1403 -0.04708 0.14655 rpy=2.0043951 0 1.57079632679
- added joint Cap_joint: type fixed, parent HeadRoll_link, child Cap, origin xyz=0 0 0 rpy=0 0 0, axis 1 0 0

File: romeo_description/urdf/romeo_generated_urdf/romeo_cap.xacro (robot description, xacro)
@@ -14,3 +14,21 @@
         <origin rpy="2.0043951 0 1.57079632679" xyz="0.1403 -0.04708 0.14655"/>
     </joint>
+    <link name="Cap">
+      <inertial>
+        <mass value="0.29923"/>
+        <inertia ixx="0.000412832" ixy="-1.67846e-06" ixz="0.000111721" iyy="0.000383921" iyz="5.04259e-05" izz="0.000264006"/>
+        <origin rpy="0 0 0" xyz="0.00 0 0.0"/>
+      </inertial>
+      <visual>
+        <geometry>
+          <mesh filename="package://romeo_description/meshes/Cap.dae" scale="1 1 1"/>
+        </geometry>
+        <origin rpy="0 0 0" xyz="0 0 0"/>
+      </visual>
+    </link>
+    <joint name="Cap_joint" type="fixed">
+        <parent link="HeadRoll_link"/>
+        <child link="Cap"/>
+        <origin rpy="0 0 1.5706" xyz="0 0 0"/>
+    </joint>
 </robot>

File: romeo_description/urdf/romeo_generated_urdf/romeo_robot.xacro (robot description, xacro)
@@ -12,4 +12,4 @@
 	<xacro:include filename="romeo_sensors.xacro"/>
 	<xacro:include filename="romeo_fingers.xacro"/>
-<!--	<xacro:include filename="romeo_cap.xacro"/> -->
+	<xacro:include filename="romeo_cap.xacro"/>
 </robot>

Commit message: remove _actuator suffix from Hand joints

File: romeo_description/urdf/romeo_generated_urdf/romeo.urdf (robot description, URDF)
Before this commit: robot romeoH37, 92 links, 91 joints
Joints:
- removed joint HeadPitch_joint
- removed joint HeadRoll_joint
- removed joint LAnklePitch_joint
- removed joint LAnkleRoll_joint
- removed joint LElbowRoll_joint
- removed joint LElbowYaw_joint
- removed joint LEyePitch_joint
- removed joint LEyeYaw_joint
- removed joint LFinger11_joint
- removed joint LFinger12_joint
- removed joint LFinger13_joint
- removed joint LFinger21_joint
- removed joint LFinger22_joint
- removed joint LFinger23_joint
- removed joint LFinger31_joint
- removed joint LFinger32_joint
- removed joint LFinger33_joint
- removed joint LHand_actuator
- removed joint LHipPitch_joint
- removed joint LHipRoll_joint
- removed joint LHipYaw_joint
- removed joint LKneePitch_joint
- removed joint LShoulderPitch_joint
- removed joint LShoulderYaw_joint
- removed joint LThumb1_joint
- removed joint LThumb2_joint
- removed joint LThumb3_joint
- removed joint LWristPitch_joint
- removed joint LWristRoll_joint
- removed joint LWristYaw_joint
- removed joint NeckPitch_joint
- removed joint NeckYaw_joint
- removed joint RAnklePitch_joint
- removed joint RAnkleRoll_joint
- removed joint RElbowRoll_joint
- removed joint RElbowYaw_joint
- removed joint REyePitch_joint
- removed joint REyeYaw_joint
- removed joint RFinger11_joint
- removed joint RFinger12_joint
- removed joint RFinger13_joint
- removed joint RFinger21_joint
- removed joint RFinger22_joint
- removed joint RFinger23_joint
- removed joint RFinger31_joint
- removed joint RFinger32_joint
- removed joint RFinger33_joint
- removed joint RHand_actuator
- removed joint RHipPitch_joint
- removed joint RHipRoll_joint
- removed joint RHipYaw_joint
- removed joint RKneePitch_joint
- removed joint RShoulderPitch_joint
- removed joint RShoulderYaw_joint
- removed joint RThumb1_joint
- removed joint RThumb2_joint
- removed joint RThumb3_joint
- removed joint RWristPitch_joint
- removed joint RWristRoll_joint
- removed joint RWristYaw_joint
- removed joint TrunkYaw_joint
- added joint HeadPitch: type revolute, parent NeckPitch_link, child HeadPitch_link, origin xyz=0 0 0.0951 rpy=0 0 0, axis 0 1.0 0, limit lower=-0.2571 upper=0.2971 effort=2.57 velocity=1.9
- added joint HeadRoll: type revolute, parent HeadPitch_link, child HeadRoll_link, origin xyz=0 0 0 rpy=0 0 0, axis 1.0 0 0, limit lower=-0.4887 upper=0.4887 effort=0.9 velocity=1.5
- added joint LAnklePitch: type revolute, parent LTibia, child LAnklePitch_link, origin xyz=0 0 -0.29 rpy=0 0 0, axis 0 1.0 0, limit lower=-0.5149 upper=0.7505 effort=25.76 velocity=2.1
- added joint LAnkleRoll: type revolute, parent LAnklePitch_link, child l_ankle, origin xyz=0 0 0 rpy=0 0 0, axis 1.0 0 0, limit lower=-0.3491 upper=0.3491 effort=25.76 velocity=2.1
- added joint LElbowRoll: type revolute, parent LShoulderYaw_link, child LForeArm, origin xyz=0.210824 7.40511e-09 -0.008631 rpy=-2.56114e-09 0 -9.31322e-09, axis 0.998889 0.0139984 0.044995, limit lower=-2.2148 upper=1.9042 effort=7.404 velocity=3.7
- added joint LElbowYaw: type revolute, parent LForeArm, child LElbow, origin xyz=0 0 0 rpy=-1.49504e-08 -1.86264e-08 2.12577e-09, axis -0.0449994 0 0.998987, limit lower=-1.5228 upper=0.0044 effort=6.02 velocity=4.0
- added joint LEyePitch: type revolute, parent LEyeYaw_link, child LEye, origin xyz=0 0 0 rpy=0 0 0, axis 0 1.0 0, limit lower=-0.349066 upper=0.349066 effort=0.01752 velocity=293.215
- added joint LEyeYaw: type revolute, parent HeadRoll_link, child LEyeYaw_link, origin xyz=0.08948 0.03192 0.05425 rpy=0 0 0, axis 0 0 1.0, limit lower=-0.523599 upper=0.523599 effort=0.01752 velocity=293.215
- added joint LFinger11: type continuous, parent l_wrist, child LFinger11_link, origin xyz=0.12385 -0.03024 0.00999 rpy=1.69304 1.5708 3.14159, axis 0 0 1.0, mimic joint=LHand multiplier=0.988205 offset=0
- added joint LFinger12: type continuous, parent LFinger11_link, child LFinger12_link, origin xyz=0 -0.0230929 -4.02331e-06 rpy=0 0 0, axis 0 0 1.0, mimic joint=LHand multiplier=0.988205 offset=0
- added joint LFinger13: type continuous, parent LFinger12_link, child LFinger13_link, origin xyz=0 -0.0230916 5.90086e-06 rpy=0 0 0, axis 0 0 1.0, mimic joint=LHand multiplier=0.988205 offset=0
- added joint LFinger21: type continuous, parent l_wrist, child LFinger21_link, origin xyz=0.12934 0 0.01499 rpy=1.5708 1.5708 3.14159, axis 0 0 1.0, mimic joint=LHand multiplier=0.988205 offset=0
- added joint LFinger22: type continuous, parent LFinger21_link, child LFinger22_link, origin xyz=0 -0.02309 0 rpy=0 0 0, axis 0 0 1.0, mimic joint=LHand multiplier=0.988205 offset=0
- added joint LFinger23: type continuous, parent LFinger22_link, child LFinger23_link, origin xyz=0 -0.02309 0 rpy=0 0 0, axis 0 0 1.0, mimic joint=LHand multiplier=0.988205 offset=0
- added joint LFinger31: type continuous, parent l_wrist, child LFinger31_link, origin xyz=0.11215 0.03024 0.00999 rpy=1.69304 -1.5708 3.14159, axis 0 0 1.0, mimic joint=LHand multiplier=0.988205 offset=0
- added joint LFinger32: type continuous, parent LFinger31_link, child LFinger32_link, origin xyz=0 0.0230928 4.02331e-06 rpy=0 0 0, axis 0 0 1.0, mimic joint=LHand multiplier=0.988205 offset=0
- added joint LFinger33: type continuous, parent LFinger32_link, child LFinger33_link, origin xyz=0 0.0230916 -5.91576e-06 rpy=0 0 0, axis 0 0 1.0, mimic joint=LHand multiplier=0.988205 offset=0
- added joint LHand: type revolute, parent l_wrist, child l_gripper, origin xyz=-0.0579412 -0.0159 -0.00260997 rpy=1.5708 0.0450146 -3.14159, axis 1.0 0 0, limit lower=0 upper=1.0 effort=0.649997 velocity=59.8925
- added joint LHipPitch: type revolute, parent LHip, child LThigh, origin xyz=0 0 0 rpy=0 0 0, axis 0 1.0 0, limit lower=-1.6581 upper=0.4014 effort=46.6 velocity=2.09
- added joint LHipRoll: type revolute, parent LHipYaw_link, child LHip, origin xyz=0 0 0 rpy=0 0 0, axis 1.0 0 0, limit lower=-0.2618 upper=0.5236 effort=46.6 velocity=2.09
- added joint LHipYaw: type revolute, parent body, child LHipYaw_link, origin xyz=0.05 0.096 -0.3375 rpy=0 0 0, axis 0 0 1.0, limit lower=-0.2618 upper=0.2618 effort=25.42 velocity=1.045
- added joint LKneePitch: type revolute, parent LThigh, child LTibia, origin xyz=0 0 -0.322 rpy=0 0 0, axis 0 1.0 0, limit lower=-0.0218 upper=1.9722 effort=38.17 velocity=6.0
- added joint LShoulderPitch: type revolute, parent torso, child LShoulder, origin xyz=0.049862 0.19 0.073851 rpy=1.49012e-08 7.45058e-09 0, axis 0.417025 0.895055 -0.15801, limit lower=-1.3491 upper=2.2462 effort=19.095 velocity=2.2
- added joint LShoulderYaw: type revolute, parent LShoulder, child LShoulderYaw_link, origin xyz=0 0 0 rpy=2.98023e-08 1.11759e-08 -5.58793e-08, axis 0.0401398 0.155542 0.987013, limit lower=-0.5768 upper=0.9242 effort=9.031 velocity=4.0
- added joint LThumb1: type continuous, parent l_wrist, child LThumb1_link, origin xyz=0.0624 -0.03131 -0.00574 rpy=-2.97779 1.21665 -3.14159, axis 0 0 1.0, mimic joint=LHand multiplier=1.74533 offset=0
- added joint LThumb2: type continuous, parent LThumb1_link, child LThumb2_link, origin xyz=0.000329241 -0.0388865 0.017011 rpy=1.13316 7.45058e-09 -1.80698, axis 0 0 1.0, mimic joint=LHand multiplier=0.988205 offset=0
- added joint LThumb3: type continuous, parent LThumb2_link, child LThumb3_link, origin xyz=0.0187362 0.0135152 5.21541e-06 rpy=-5.96047e-08 0 1.49012e-08, axis 0 0 1.0, mimic joint=LHand multiplier=0.988205 offset=0
- added joint LWristPitch: type revolute, parent LWristYaw_link, child l_wrist, origin xyz=0 0 0 rpy=0 0 0, axis 0 1.0 0, limit lower=-0.988 upper=0.8969 effort=0.6 velocity=3.75
- added joint LWristRoll: type revolute, parent LElbow, child LWristRoll_link, origin xyz=0.190404 0 0.008631 rpy=0 -7.45058e-09 0, axis 0.998987 0 0.0449994, limit lower=-3.6303 upper=0.4887 effort=2.177 velocity=1.1
- added joint LWristYaw: type revolute, parent LWristRoll_link, child LWristYaw_link, origin xyz=0 0 0 rpy=0 0 0, axis -0.0449994 0 0.998987, limit lower=-0.4014 upper=0.4014 effort=0.862 velocity=2.26
- added joint NeckPitch: type revolute, parent NeckYaw_link, child NeckPitch_link, origin xyz=0 0 0 rpy=0 -2.98023e-08 0, axis 0 1.0 0, limit lower=-0.3142 upper=0.6632 effort=2.978 velocity=2.2
- added joint NeckYaw: type revolute, parent torso, child NeckYaw_link, origin xyz=0.0548 0 0.1675 rpy=0 -2.98023e-08 0, axis 0.173651 0 0.984807, limit lower=-2.0595 upper=2.0595 effort=3.662 velocity=4.0
- added joint RAnklePitch: type revolute, parent RTibia, child RAnklePitch_link, origin xyz=0 0 -0.29 rpy=0 0 0, axis 0 1.0 0, limit lower=-0.5149 upper=0.7505 effort=25.76 velocity=2.1
- added joint RAnkleRoll: type revolute, parent RAnklePitch_link, child r_ankle, origin xyz=0 0 0 rpy=0 0 0, axis 1.0 0 0, limit lower=-0.3491 upper=0.3491 effort=25.76 velocity=2.1
- added joint RElbowRoll: type revolute, parent RShoulderYaw_link, child RForeArm, origin xyz=0.210824 -1.48548e-08 -0.008631 rpy=6.69388e-09 7.45058e-09 -7.91624e-08, axis 0.998889 -0.0139984 0.044995, limit lower=-1.9047 upper=2.2143 effort=7.404 velocity=3.7
- added joint RElbowYaw: type revolute, parent RForeArm, child RElbow, origin xyz=0 0 0 rpy=1.49504e-08 -1.86264e-08 -2.12577e-09, axis -0.0449994 0 0.998987, limit lower=-0.0047 upper=1.5225 effort=6.02 velocity=4.0
- added joint REyePitch: type revolute, parent REyeYaw_link, child REye, origin xyz=0 0 0 rpy=0 0 0, axis 0 1.0 0, limit lower=-0.349066 upper=0.349066 effort=0.01752 velocity=293.215
- added joint REyeYaw: type revolute, parent HeadRoll_link, child REyeYaw_link, origin xyz=0.08948 -0.03192 0.05425 rpy=0 0 0, axis 0 0 1.0, limit lower=-0.523599 upper=0.523599 effort=0.01752 velocity=293.215
- added joint RFinger11: type continuous, parent r_wrist, child RFinger11_link, origin xyz=0.12385 0.03024 0.00999 rpy=1.69304 -1.5708 3.14159, axis 0 0 1.0, mimic joint=RHand multiplier=0.988205 offset=0
- added joint RFinger12: type continuous, parent RFinger11_link, child RFinger12_link, origin xyz=0 0.0230929 4.02331e-06 rpy=0 0 0, axis 0 0 1.0, mimic joint=RHand multiplier=0.988205 offset=0
- added joint RFinger13: type continuous, parent RFinger12_link, child RFinger13_link, origin xyz=0 0.0230916 -5.90086e-06 rpy=0 0 0, axis 0 0 1.0, mimic joint=RHand multiplier=0.988205 offset=0
- added joint RFinger21: type continuous, parent r_wrist, child RFinger21_link, origin xyz=0.12934 0 0.01499 rpy=1.5708 -1.5708 -3.14159, axis 0 0 1.0, mimic joint=RHand multiplier=0.988205 offset=0
- added joint RFinger22: type continuous, parent RFinger21_link, child RFinger22_link, origin xyz=0 0.02309 0 rpy=0 0 0, axis 0 0 1.0, mimic joint=RHand multiplier=0.988205 offset=0
- added joint RFinger23: type continuous, parent RFinger22_link, child RFinger23_link, origin xyz=0 0.02309 0 rpy=0 0 0, axis 0 0 1.0, mimic joint=RHand multiplier=0.988205 offset=0
- added joint RFinger31: type continuous, parent r_wrist, child RFinger31_link, origin xyz=0.11215 -0.03024 0.00999 rpy=1.69304 1.5708 3.14159, axis 0 0 1.0, mimic joint=RHand multiplier=0.988205 offset=0
- added joint RFinger32: type continuous, parent RFinger31_link, child RFinger32_link, origin xyz=0 -0.0230929 -4.02331e-06 rpy=0 0 0, axis 0 0 1.0, mimic joint=RHand multiplier=0.988205 offset=0
- added joint RFinger33: type continuous, parent RFinger32_link, child RFinger33_link, origin xyz=0 -0.0230916 5.90086e-06 rpy=0 0 0, axis 0 0 1.0, mimic joint=RHand multiplier=0.988205 offset=0
- added joint RHand: type revolute, parent r_wrist, child r_gripper, origin xyz=-0.0579412 -0.0159 -0.00260997 rpy=1.5708 0.0450146 -3.14159, axis 1.0 0 0, limit lower=0 upper=1.0 effort=0.649997 velocity=59.8925
- added joint RHipPitch: type revolute, parent RHip, child RThigh, origin xyz=0 0 0 rpy=0 0 0, axis 0 1.0 0, limit lower=-1.6581 upper=0.4014 effort=46.6 velocity=2.09
- added joint RHipRoll: type revolute, parent RHipYaw_link, child RHip, origin xyz=0 0 0 rpy=0 0 0, axis 1.0 0 0, limit lower=-0.5236 upper=0.2618 effort=46.6 velocity=2.09
- added joint RHipYaw: type revolute, parent body, child RHipYaw_link, origin xyz=0.05 -0.096 -0.3375 rpy=0 0 0, axis 0 0 1.0, limit lower=-0.2618 upper=0.2618 effort=25.42 velocity=1.045
- added joint RKneePitch: type revolute, parent RThigh, child RTibia, origin xyz=0 0 -0.322 rpy=0 0 0, axis 0 1.0 0, limit lower=-0.0218 upper=1.9722 effort=38.17 velocity=6.0
- added joint RShoulderPitch: type revolute, parent torso, child RShoulder, origin xyz=0.049862 -0.19 0.073851 rpy=-1.49012e-08 7.45058e-09 0, axis -0.417025 0.895055 0.15801, limit lower=-1.4554 upper=2.1399 effort=19.095 velocity=2.2
- added joint RShoulderYaw: type revolute, parent RShoulder, child RShoulderYaw_link, origin xyz=0 0 0 rpy=-2.98023e-08 1.49012e-08 -6.42613e-08, axis 0.0401398 -0.155542 0.987014, limit lower=-1.0985 upper=0.4025 effort=9.031 velocity=4.0
- added joint RThumb1: type continuous, parent r_wrist, child RThumb1_link, origin xyz=0.0624 0.03131 -0.00574 rpy=0.1638 -1.21665 0, axis 0 0 1.0, mimic joint=RHand multiplier=1.74533 offset=0
- added joint RThumb2: type continuous, parent RThumb1_link, child RThumb2_link, origin xyz=-0.000329241 0.0388865 -0.017011 rpy=1.13316 0 -1.80698, axis 0 0 1.0, mimic joint=RHand multiplier=0.988205 offset=0
- added joint RThumb3: type continuous, parent RThumb2_link, child RThumb3_link, origin xyz=-0.0187362 -0.0135152 -5.21541e-06 rpy=-5.96047e-08 -1.49012e-08 1.49012e-08, axis 0 0 1.0, mimic joint=RHand multiplier=0.988205 offset=0
- added joint RWristPitch: type revolute, parent RWristYaw_link, child r_wrist, origin xyz=0 0 0 rpy=0 0 0, axis 0 1.0 0, limit lower=-0.9868 upper=0.8981 effort=0.6 velocity=3.75
- added joint RWristRoll: type revolute, parent RElbow, child RWristRoll_link, origin xyz=0.190404 0 0.008631 rpy=0 -7.45058e-09 0, axis 0.998987 0 0.0449994, limit lower=-0.4887 upper=3.6303 effort=2.177 velocity=1.1
- added joint RWristYaw: type revolute, parent RWristRoll_link, child RWristYaw_link, origin xyz=0 0 0 rpy=0 0 0, axis -0.0449994 0 0.998987, limit lower=-0.4014 upper=0.4014 effort=0.862 velocity=2.26
- added joint TrunkYaw: type revolute, parent torso, child body, origin xyz=0 0 0 rpy=0 0 0, axis 0 0 1.0, limit lower=-0.7575 upper=0.7575 effort=80.902 velocity=1.5
- joint Cap_joint: axis 1 0 0 -> (none)

File: romeo_description/urdf/romeo_generated_urdf/romeo_arms.xacro (robot description, xacro)
@@ -4,5 +4,5 @@
  *********************************************************************-->
 <robot xmlns:xacro="http://www.ros.org/wiki/xacro">
-	<joint name="LShoulderPitch_joint" type="revolute">
+	<joint name="LShoulderPitch" type="revolute">
 		<parent link="torso"/>
 		<child link="LShoulder"/>
@@ -18,5 +18,5 @@
 		</inertial>
 	</link>
-	<joint name="LShoulderYaw_joint" type="revolute">
+	<joint name="LShoulderYaw" type="revolute">
 		<parent link="LShoulder"/>
 		<child link="LShoulderYaw_link"/>
@@ -33,5 +33,5 @@
 		<xacro:insert_visu_LShoulderYaw_link/>
 	</link>
-	<joint name="LElbowRoll_joint" type="revolute">
+	<joint name="LElbowRoll" type="revolute">
 		<parent link="LShoulderYaw_link"/>
 		<child link="LForeArm"/>
@@ -47,5 +47,5 @@
 		</inertial>
 	</link>
-	<joint name="LElbowYaw_joint" type="revolute">
+	<joint name="LElbowYaw" type="revolute">
 		<parent link="LForeArm"/>
 		<child link="LElbow"/>
@@ -62,5 +62,5 @@
 		<xacro:insert_visu_LElbow/>
 	</link>
-	<joint name="LWristRoll_joint" type="revolute">
+	<joint name="LWristRoll" type="revolute">
 		<parent link="LElbow"/>
 		<child link="LWristRoll_link"/>
@@ -77,5 +77,5 @@
 		<xacro:insert_visu_LWristRoll_link/>
 	</link>
-	<joint name="LWristYaw_joint" type="revolute">
+	<joint name="LWristYaw" type="revolute">
 		<parent link="LWristRoll_link"/>
 		<child link="LWristYaw_link"/>
@@ -92,5 +92,5 @@
 		<xacro:insert_visu_LWristYaw_link/>
 	</link>
-	<joint name="LWristPitch_joint" type="revolute">
+	<joint name="LWristPitch" type="revolute">
 		<parent link="LWristYaw_link"/>
 		<child link="l_wrist"/>
@@ -107,5 +107,5 @@
 		<xacro:insert_visu_l_wrist/>
 	</link>
-	<joint name="LHand_actuator" type="revolute">
+	<joint name="LHand" type="revolute">
 		<parent link="l_wrist"/>
 		<child link="l_gripper"/>
@@ -115,5 +115,5 @@
 	</joint>
 	<link name="l_gripper"/>
-	<joint name="RShoulderPitch_joint" type="revolute">
+	<joint name="RShoulderPitch" type="revolute">
 		<parent link="torso"/>
 		<child link="RShoulder"/>
@@ -129,5 +129,5 @@
 		</inertial>
 	</link>
-	<joint name="RShoulderYaw_joint" type="revolute">
+	<joint name="RShoulderYaw" type="revolute">
 		<parent link="RShoulder"/>
 		<child link="RShoulderYaw_link"/>
@@ -144,5 +144,5 @@
 		<xacro:insert_visu_RShoulderYaw_link/>
 	</link>
-	<joint name="RElbowRoll_joint" type="revolute">
+	<joint name="RElbowRoll" type="revolute">
 		<parent link="RShoulderYaw_link"/>
 		<child link="RForeArm"/>
@@ -158,5 +158,5 @@
 		</inertial>
 	</link>
-	<joint name="RElbowYaw_joint" type="revolute">
+	<joint name="RElbowYaw" type="revolute">
 		<parent link="RForeArm"/>
 		<child link="RElbow"/>
@@ -173,5 +173,5 @@
 		<xacro:insert_visu_RElbow/>
 	</link>
-	<joint name="RWristRoll_joint" type="revolute">
+	<joint name="RWristRoll" type="revolute">
 		<parent link="RElbow"/>
 		<child link="RWristRoll_link"/>
@@ -188,5 +188,5 @@
 		<xacro:insert_visu_RWristRoll_link/>
 	</link>
-	<joint name="RWristYaw_joint" type="revolute">
+	<joint name="RWristYaw" type="revolute">
 		<parent link="RWristRoll_link"/>
 		<child link="RWristYaw_link"/>
@@ -203,5 +203,5 @@
 		<xacro:insert_visu_RWristYaw_link/>
 	</link>
-	<joint name="RWristPitch_joint" type="revolute">
+	<joint name="RWristPitch" type="revolute">
 		<parent link="RWristYaw_link"/>
 		<child link="r_wrist"/>
@@ -218,5 +218,5 @@
 		<xacro:insert_visu_r_wrist/>
 	</link>
-	<joint name="RHand_actuator" type="revolute">
+	<joint name="RHand" type="revolute">
 		<parent link="r_wrist"/>
 		<child link="r_gripper"/>

File: romeo_description/urdf/romeo_generated_urdf/romeo_cap.xacro (robot description, xacro)
@@ -18,5 +18,5 @@
         <mass value="0.29923"/>
         <inertia ixx="0.000412832" ixy="-1.67846e-06" ixz="0.000111721" iyy="0.000383921" iyz="5.04259e-05" izz="0.000264006"/>
-        <origin rpy="0 0 0" xyz="0.00 0 0.0"/>
+        <origin rpy="0 0 0" xyz="0 0 0"/>
       </inertial>
       <visual>
@@ -30,5 +30,5 @@
         <parent link="HeadRoll_link"/>
         <child link="Cap"/>
-        <origin rpy="0 0 1.5706" xyz="0 0 0"/>
+        <origin rpy="0 0 0" xyz="0 0 0"/>
     </joint>
 </robot>

File: romeo_description/urdf/romeo_generated_urdf/romeo_eyes.xacro (robot description, xacro)
@@ -4,5 +4,5 @@
  *********************************************************************-->
 <robot xmlns:xacro="http://www.ros.org/wiki/xacro">
-	<joint name="LEyeYaw_joint" type="revolute">
+	<joint name="LEyeYaw" type="revolute">
 		<parent link="HeadRoll_link"/>
 		<child link="LEyeYaw_link"/>
@@ -18,5 +18,5 @@
 		</inertial>
 	</link>
-	<joint name="LEyePitch_joint" type="revolute">
+	<joint name="LEyePitch" type="revolute">
 		<parent link="LEyeYaw_link"/>
 		<child link="LEye"/>
@@ -33,5 +33,5 @@
 		<xacro:insert_visu_LEye/>
 	</link>
-	<joint name="REyeYaw_joint" type="revolute">
+	<joint name="REyeYaw" type="revolute">
 		<parent link="HeadRoll_link"/>
 		<child link="REyeYaw_link"/>
@@ -47,5 +47,5 @@
 		</inertial>
 	</link>
-	<joint name="REyePitch_joint" type="revolute">
+	<joint name="REyePitch" type="revolute">
 		<parent link="REyeYaw_link"/>
 		<child link="REye"/>
