Commit message: remove _actuator suffix from Hand joints

File: romeo_description/urdf/romeo_generated_urdf/romeo_fingers.xacro (robot description, xacro)
@@ -7,240 +7,240 @@
 		<xacro:insert_visu_RFinger13_link/>
 	</link>
-	<joint name="RFinger13_joint" type="continuous">
+	<joint name="RFinger13" type="continuous">
 		<parent link="RFinger12_link"/>
 		<child link="RFinger13_link"/>
 		<origin rpy="0 0 0" xyz="0 0.0230916 -5.90086e-06"/>
 		<axis xyz="0 0 1.0"/>
-		<mimic joint="RHand_actuator" multiplier="0.988205" offset="0"/>
+		<mimic joint="RHand" multiplier="0.988205" offset="0"/>
 	</joint>
 	<link name="RFinger12_link">
 		<xacro:insert_visu_RFinger12_link/>
 	</link>
-	<joint name="RFinger12_joint" type="continuous">
+	<joint name="RFinger12" type="continuous">
 		<parent link="RFinger11_link"/>
 		<child link="RFinger12_link"/>
 		<origin rpy="0 0 0" xyz="0 0.0230929 4.02331e-06"/>
 		<axis xyz="0 0 1.0"/>
-		<mimic joint="RHand_actuator" multiplier="0.988205" offset="0"/>
+		<mimic joint="RHand" multiplier="0.988205" offset="0"/>
 	</joint>
 	<link name="LFinger33_link">
 		<xacro:insert_visu_LFinger33_link/>
 	</link>
-	<joint name="LFinger33_joint" type="continuous">
+	<joint name="LFinger33" type="continuous">
 		<parent link="LFinger32_link"/>
 		<child link="LFinger33_link"/>
 		<origin rpy="0 0 0" xyz="0 0.0230916 -5.91576e-06"/>
 		<axis xyz="0 0 1.0"/>
-		<mimic joint="LHand_actuator" multiplier="0.988205" offset="0"/>
+		<mimic joint="LHand" multiplier="0.988205" offset="0"/>
 	</joint>
 	<link name="RFinger31_link">
 		<xacro:insert_visu_RFinger31_link/>
 	</link>
-	<joint name="RFinger31_joint" type="continuous">
+	<joint name="RFinger31" type="continuous">
 		<parent link="r_wrist"/>
 		<child link="RFinger31_link"/>
 		<origin rpy="1.69304 1.5708 3.14159" xyz="0.11215 -0.03024 0.00999"/>
 		<axis xyz="0 0 1.0"/>
-		<mimic joint="RHand_actuator" multiplier="0.988205" offset="0"/>
+		<mimic joint="RHand" multiplier="0.988205" offset="0"/>
 	</joint>
 	<link name="RFinger32_link">
 		<xacro:insert_visu_RFinger32_link/>
 	</link>
-	<joint name="RFinger32_joint" type="continuous">
+	<joint name="RFinger32" type="continuous">
 		<parent link="RFinger31_link"/>
 		<child link="RFinger32_link"/>
 		<origin rpy="0 0 0" xyz="0 -0.0230929 -4.02331e-06"/>
 		<axis xyz="0 0 1.0"/>
-		<mimic joint="RHand_actuator" multiplier="0.988205" offset="0"/>
+		<mimic joint="RHand" multiplier="0.988205" offset="0"/>
 	</joint>
 	<link name="LFinger21_link">
 		<xacro:insert_visu_LFinger21_link/>
 	</link>
-	<joint name="LFinger21_joint" type="continuous">
+	<joint name="LFinger21" type="continuous">
 		<parent link="l_wrist"/>
 		<child link="LFinger21_link"/>
 		<origin rpy="1.5708 1.5708 3.14159" xyz="0.12934 0 0.01499"/>
 		<axis xyz="0 0 1.0"/>
-		<mimic joint="LHand_actuator" multiplier="0.988205" offset="0"/>
+		<mimic joint="LHand" multiplier="0.988205" offset="0"/>
 	</joint>
 	<link name="LFinger13_link">
 		<xacro:insert_visu_LFinger13_link/>
 	</link>
-	<joint name="LFinger13_joint" type="continuous">
+	<joint name="LFinger13" type="continuous">
 		<parent link="LFinger12_link"/>
 		<child link="LFinger13_link"/>
 		<origin rpy="0 0 0" xyz="0 -0.0230916 5.90086e-06"/>
 		<axis xyz="0 0 1.0"/>
-		<mimic joint="LHand_actuator" multiplier="0.988205" offset="0"/>
+		<mimic joint="LHand" multiplier="0.988205" offset="0"/>
 	</joint>
 	<link name="LFinger32_link">
 		<xacro:insert_visu_LFinger32_link/>
 	</link>
-	<joint name="LFinger32_joint" type="continuous">
+	<joint name="LFinger32" type="continuous">
 		<parent link="LFinger31_link"/>
 		<child link="LFinger32_link"/>
 		<origin rpy="0 0 0" xyz="0 0.0230928 4.02331e-06"/>
 		<axis xyz="0 0 1.0"/>
-		<mimic joint="LHand_actuator" multiplier="0.988205" offset="0"/>
+		<mimic joint="LHand" multiplier="0.988205" offset="0"/>
 	</joint>
 	<link name="LFinger11_link">
 		<xacro:insert_visu_LFinger11_link/>
 	</link>
-	<joint name="LFinger11_joint" type="continuous">
+	<joint name="LFinger11" type="continuous">
 		<parent link="l_wrist"/>
 		<child link="LFinger11_link"/>
 		<origin rpy="1.69304 1.5708 3.14159" xyz="0.12385 -0.03024 0.00999"/>
 		<axis xyz="0 0 1.0"/>
-		<mimic joint="LHand_actuator" multiplier="0.988205" offset="0"/>
+		<mimic joint="LHand" multiplier="0.988205" offset="0"/>
 	</joint>
 	<link name="RFinger22_link">
 		<xacro:insert_visu_RFinger22_link/>
 	</link>
-	<joint name="RFinger22_joint" type="continuous">
+	<joint name="RFinger22" type="continuous">
 		<parent link="RFinger21_link"/>
 		<child link="RFinger22_link"/>
 		<origin rpy="0 0 0" xyz="0 0.02309 0"/>
 		<axis xyz="0 0 1.0"/>
-		<mimic joint="RHand_actuator" multiplier="0.988205" offset="0"/>
+		<mimic joint="RHand" multiplier="0.988205" offset="0"/>
 	</joint>
 	<link name="LFinger22_link">
 		<xacro:insert_visu_LFinger22_link/>
 	</link>
-	<joint name="LFinger22_joint" type="continuous">
+	<joint name="LFinger22" type="continuous">
 		<parent link="LFinger21_link"/>
 		<child link="LFinger22_link"/>
 		<origin rpy="0 0 0" xyz="0 -0.02309 0"/>
 		<axis xyz="0 0 1.0"/>
-		<mimic joint="LHand_actuator" multiplier="0.988205" offset="0"/>
+		<mimic joint="LHand" multiplier="0.988205" offset="0"/>
 	</joint>
 	<link name="RFinger21_link">
 		<xacro:insert_visu_RFinger21_link/>
 	</link>
-	<joint name="RFinger21_joint" type="continuous">
+	<joint name="RFinger21" type="continuous">
 		<parent link="r_wrist"/>
 		<child link="RFinger21_link"/>
 		<origin rpy="1.5708 -1.5708 -3.14159" xyz="0.12934 0 0.01499"/>
 		<axis xyz="0 0 1.0"/>
-		<mimic joint="RHand_actuator" multiplier="0.988205" offset="0"/>
+		<mimic joint="RHand" multiplier="0.988205" offset="0"/>
 	</joint>
 	<link name="LFinger12_link">
 		<xacro:insert_visu_LFinger12_link/>
 	</link>
-	<joint name="LFinger12_joint" type="continuous">
+	<joint name="LFinger12" type="continuous">
 		<parent link="LFinger11_link"/>
 		<child link="LFinger12_link"/>
 		<origin rpy="0 0 0" xyz="0 -0.0230929 -4.02331e-06"/>
 		<axis xyz="0 0 1.0"/>
-		<mimic joint="LHand_actuator" multiplier="0.988205" offset="0"/>
+		<mimic joint="LHand" multiplier="0.988205" offset="0"/>
 	</joint>
 	<link name="RFinger23_link">
 		<xacro:insert_visu_RFinger23_link/>
 	</link>
-	<joint name="RFinger23_joint" type="continuous">
+	<joint name="RFinger23" type="continuous">
 		<parent link="RFinger22_link"/>
 		<child link="RFinger23_link"/>
 		<origin rpy="0 0 0" xyz="0 0.02309 0"/>
 		<axis xyz="0 0 1.0"/>
-		<mimic joint="RHand_actuator" multiplier="0.988205" offset="0"/>
+		<mimic joint="RHand" multiplier="0.988205" offset="0"/>
 	</joint>
 	<link name="RFinger11_link">
 		<xacro:insert_visu_RFinger11_link/>
 	</link>
-	<joint name="RFinger11_joint" type="continuous">
+	<joint name="RFinger11" type="continuous">
 		<parent link="r_wrist"/>
 		<child link="RFinger11_link"/>
 		<origin rpy="1.69304 -1.5708 3.14159" xyz="0.12385 0.03024 0.00999"/>
 		<axis xyz="0 0 1.0"/>
-		<mimic joint="RHand_actuator" multiplier="0.988205" offset="0"/>
+		<mimic joint="RHand" multiplier="0.988205" offset="0"/>
 	</joint>
 	<link name="LFinger23_link">
 		<xacro:insert_visu_LFinger23_link/>
 	</link>
-	<joint name="LFinger23_joint" type="continuous">
+	<joint name="LFinger23" type="continuous">
 		<parent link="LFinger22_link"/>
 		<child link="LFinger23_link"/>
 		<origin rpy="0 0 0" xyz="0 -0.02309 0"/>
 		<axis xyz="0 0 1.0"/>
-		<mimic joint="LHand_actuator" multiplier="0.988205" offset="0"/>
+		<mimic joint="LHand" multiplier="0.988205" offset="0"/>
 	</joint>
 	<link name="LFinger31_link">
 		<xacro:insert_visu_LFinger31_link/>
 	</link>
-	<joint name="LFinger31_joint" type="continuous">
+	<joint name="LFinger31" type="continuous">
 		<parent link="l_wrist"/>
 		<child link="LFinger31_link"/>
 		<origin rpy="1.69304 -1.5708 3.14159" xyz="0.11215 0.03024 0.00999"/>
 		<axis xyz="0 0 1.0"/>
-		<mimic joint="LHand_actuator" multiplier="0.988205" offset="0"/>
+		<mimic joint="LHand" multiplier="0.988205" offset="0"/>
 	</joint>
 	<link name="RFinger33_link">
 		<xacro:insert_visu_RFinger33_link/>
 	</link>
-	<joint name="RFinger33_joint" type="continuous">
+	<joint name="RFinger33" type="continuous">
 		<parent link="RFinger32_link"/>
 		<child link="RFinger33_link"/>
 		<origin rpy="0 0 0" xyz="0 -0.0230916 5.90086e-06"/>
 		<axis xyz="0 0 1.0"/>
-		<mimic joint="RHand_actuator" multiplier="0.988205" offset="0"/>
+		<mimic joint="RHand" multiplier="0.988205" offset="0"/>
 	</joint>
 	<link name="LThumb3_link">
 		<xacro:insert_visu_LThumb3_link/>
 	</link>
-	<joint name="LThumb3_joint" type="continuous">
+	<joint name="LThumb3" type="continuous">
 		<parent link="LThumb2_link"/>
 		<child link="LThumb3_link"/>
 		<origin rpy="-5.96047e-08 0 1.49012e-08" xyz="0.0187362 0.0135152 5.21541e-06"/>
 		<axis xyz="0 0 1.0"/>
-		<mimic joint="LHand_actuator" multiplier="0.988205" offset="0"/>
+		<mimic joint="LHand" multiplier="0.988205" offset="0"/>
 	</joint>
 	<link name="LThumb1_link">
 		<xacro:insert_visu_LThumb1_link/>
 	</link>
-	<joint name="LThumb1_joint" type="continuous">
+	<joint name="LThumb1" type="continuous">
 		<parent link="l_wrist"/>
 		<child link="LThumb1_link"/>
 		<origin rpy="-2.97779 1.21665 -3.14159" xyz="0.0624 -0.03131 -0.00574"/>
 		<axis xyz="0 0 1.0"/>
-		<mimic joint="LHand_actuator" multiplier="1.74533" offset="0"/>
+		<mimic joint="LHand" multiplier="1.74533" offset="0"/>
 	</joint>
 	<link name="RThumb1_link">
 		<xacro:insert_visu_RThumb1_link/>
 	</link>
-	<joint name="RThumb1_joint" type="continuous">
+	<joint name="RThumb1" type="continuous">
 		<parent link="r_wrist"/>
 		<child link="RThumb1_link"/>
 		<origin rpy="0.1638 -1.21665 0" xyz="0.0624 0.03131 -0.00574"/>
 		<axis xyz="0 0 1.0"/>
-		<mimic joint="RHand_actuator" multiplier="1.74533" offset="0"/>
+		<mimic joint="RHand" multiplier="1.74533" offset="0"/>
 	</joint>
 	<link name="RThumb2_link">
 		<xacro:insert_visu_RThumb2_link/>
 	</link>
-	<joint name="RThumb2_joint" type="continuous">
+	<joint name="RThumb2" type="continuous">
 		<parent link="RThumb1_link"/>
 		<child link="RThumb2_link"/>
 		<origin rpy="1.13316 0 -1.80698" xyz="-0.000329241 0.0388865 -0.017011"/>
 		<axis xyz="0 0 1.0"/>
-		<mimic joint="RHand_actuator" multiplier="0.988205" offset="0"/>
+		<mimic joint="RHand" multiplier="0.988205" offset="0"/>
 	</joint>
 	<link name="LThumb2_link">
 		<xacro:insert_visu_LThumb2_link/>
 	</link>
-	<joint name="LThumb2_joint" type="continuous">
+	<joint name="LThumb2" type="continuous">
 		<parent link="LThumb1_link"/>
 		<child link="LThumb2_link"/>
 		<origin rpy="1.13316 7.45058e-09 -1.80698" xyz="0.000329241 -0.0388865 0.017011"/>
 		<axis xyz="0 0 1.0"/>
-		<mimic joint="LHand_actuator" multiplier="0.988205" offset="0"/>
+		<mimic joint="LHand" multiplier="0.988205" offset="0"/>
 	</joint>
 	<link name="RThumb3_link">
 		<xacro:insert_visu_RThumb3_link/>
 	</link>
-	<joint name="RThumb3_joint" type="continuous">
+	<joint name="RThumb3" type="continuous">
 		<parent link="RThumb2_link"/>
 		<child link="RThumb3_link"/>
 		<origin rpy="-5.96047e-08 -1.49012e-08 1.49012e-08" xyz="-0.0187362 -0.0135152 -5.21541e-06"/>
 		<axis xyz="0 0 1.0"/>
-		<mimic joint="RHand_actuator" multiplier="0.988205" offset="0"/>
+		<mimic joint="RHand" multiplier="0.988205" offset="0"/>
 	</joint>
 </robot>

File: romeo_description/urdf/romeo_generated_urdf/romeo_head.xacro (robot description, xacro)
@@ -4,5 +4,5 @@
  *********************************************************************-->
 <robot xmlns:xacro="http://www.ros.org/wiki/xacro">
-	<joint name="NeckYaw_joint" type="revolute">
+	<joint name="NeckYaw" type="revolute">
 		<parent link="torso"/>
 		<child link="NeckYaw_link"/>
@@ -18,5 +18,5 @@
 		</inertial>
 	</link>
-	<joint name="NeckPitch_joint" type="revolute">
+	<joint name="NeckPitch" type="revolute">
 		<parent link="NeckYaw_link"/>
 		<child link="NeckPitch_link"/>
@@ -33,5 +33,5 @@
 		<xacro:insert_visu_NeckPitch_link/>
 	</link>
-	<joint name="HeadPitch_joint" type="revolute">
+	<joint name="HeadPitch" type="revolute">
 		<parent link="NeckPitch_link"/>
 		<child link="HeadPitch_link"/>
@@ -47,5 +47,5 @@
 		</inertial>
 	</link>
-	<joint name="HeadRoll_joint" type="revolute">
+	<joint name="HeadRoll" type="revolute">
 		<parent link="HeadPitch_link"/>
 		<child link="HeadRoll_link"/>

File: romeo_description/urdf/romeo_generated_urdf/romeo_legs.xacro (robot description, xacro)
@@ -4,5 +4,5 @@
  *********************************************************************-->
 <robot xmlns:xacro="http://www.ros.org/wiki/xacro">
-	<joint name="LHipYaw_joint" type="revolute">
+	<joint name="LHipYaw" type="revolute">
 		<parent link="body"/>
 		<child link="LHipYaw_link"/>
@@ -18,5 +18,5 @@
 		</inertial>
 	</link>
-	<joint name="LHipRoll_joint" type="revolute">
+	<joint name="LHipRoll" type="revolute">
 		<parent link="LHipYaw_link"/>
 		<child link="LHip"/>
@@ -32,5 +32,5 @@
 		</inertial>
 	</link>
-	<joint name="LHipPitch_joint" type="revolute">
+	<joint name="LHipPitch" type="revolute">
 		<parent link="LHip"/>
 		<child link="LThigh"/>
@@ -47,5 +47,5 @@
 		<xacro:insert_visu_LThigh/>
 	</link>
-	<joint name="LKneePitch_joint" type="revolute">
+	<joint name="LKneePitch" type="revolute">
 		<parent link="LThigh"/>
 		<child link="LTibia"/>
@@ -62,5 +62,5 @@
 		<xacro:insert_visu_LTibia/>
 	</link>
-	<joint name="LAnklePitch_joint" type="revolute">
+	<joint name="LAnklePitch" type="revolute">
 		<parent link="LTibia"/>
 		<child link="LAnklePitch_link"/>
@@ -76,5 +76,5 @@
 		</inertial>
 	</link>
-	<joint name="LAnkleRoll_joint" type="revolute">
+	<joint name="LAnkleRoll" type="revolute">
 		<parent link="LAnklePitch_link"/>
 		<child link="l_ankle"/>
@@ -98,5 +98,5 @@
 	</joint>
 	<link name="l_sole"/>
-	<joint name="RHipYaw_joint" type="revolute">
+	<joint name="RHipYaw" type="revolute">
 		<parent link="body"/>
 		<child link="RHipYaw_link"/>
@@ -112,5 +112,5 @@
 		</inertial>
 	</link>
-	<joint name="RHipRoll_joint" type="revolute">
+	<joint name="RHipRoll" type="revolute">
 		<parent link="RHipYaw_link"/>
 		<child link="RHip"/>
@@ -126,5 +126,5 @@
 		</inertial>
 	</link>
-	<joint name="RHipPitch_joint" type="revolute">
+	<joint name="RHipPitch" type="revolute">
 		<parent link="RHip"/>
 		<child link="RThigh"/>
@@ -141,5 +141,5 @@
 		<xacro:insert_visu_RThigh/>
 	</link>
-	<joint name="RKneePitch_joint" type="revolute">
+	<joint name="RKneePitch" type="revolute">
 		<parent link="RThigh"/>
 		<child link="RTibia"/>
@@ -156,5 +156,5 @@
 		<xacro:insert_visu_RTibia/>
 	</link>
-	<joint name="RAnklePitch_joint" type="revolute">
+	<joint name="RAnklePitch" type="revolute">
 		<parent link="RTibia"/>
 		<child link="RAnklePitch_link"/>
@@ -170,5 +170,5 @@
 		</inertial>
 	</link>
-	<joint name="RAnkleRoll_joint" type="revolute">
+	<joint name="RAnkleRoll" type="revolute">
 		<parent link="RAnklePitch_link"/>
 		<child link="r_ankle"/>

File: romeo_description/urdf/romeo_generated_urdf/romeo_robot.xacro (robot description, xacro)
@@ -12,4 +12,4 @@
 	<xacro:include filename="romeo_sensors.xacro"/>
 	<xacro:include filename="romeo_fingers.xacro"/>
-	<xacro:include filename="romeo_cap.xacro"/>
+    <xacro:include filename="romeo_cap.xacro"/>
 </robot>

File: romeo_description/urdf/romeo_generated_urdf/romeo_torso.xacro (robot description, xacro)
@@ -19,5 +19,5 @@
 		<xacro:insert_visu_torso/>
 	</link>
-	<joint name="TrunkYaw_joint" type="revolute">
+	<joint name="TrunkYaw" type="revolute">
 		<parent link="torso"/>
 		<child link="body"/>

Commit message: do not forget the cap

File: romeo_description/urdf/romeo_generated_urdf/romeo.urdf (robot description, URDF)
Before this commit: robot romeoH37, 94 links, 93 joints
Links:
- added link CameraDepth_frame
- added link Cap, mass 0.29923; visual mesh filename=package://romeo_description/meshes/Cap.dae scale=1 1 1
Joints:
- added joint CameraDepth_joint: type fixed, parent HeadRoll_link, child CameraDepth_frame, origin xyz=0.1403 -0.04708 0.14655 rpy=2.0043951 0 1.57079632679
- added joint Cap_joint: type fixed, parent HeadRoll_link, child Cap, origin xyz=0 0 0 rpy=0 0 0

File: romeo_description/urdf/romeo_generated_urdf/romeo_robot.xacro (robot description, xacro)
@@ -12,3 +12,4 @@
 	<xacro:include filename="romeo_sensors.xacro"/>
 	<xacro:include filename="romeo_fingers.xacro"/>
+	<xacro:include filename="romeo_cap.xacro"/>
 </robot>
