Commit message: update to the latest Romeo URDF

File: romeo_description/urdf/romeo_generated_urdf/romeo.urdf (robot description, URDF)
Before this commit: robot romeoH37, 96 links, 95 joints
Links:
- link HeadPitch_link: mass 0.13728 -> 0.158407
- link HeadRoll_link: mass 1.79432 -> 2.07047
- link LAnklePitch_link: mass 0.42803 -> 0.464512
- link LElbow: mass 0.36997 -> 0.460203
- link LForeArm: mass 0.48271 -> 0.600439
- link LHip: mass 0.65864 -> 0.714778
- link LHipYaw_link: mass 0.51527 -> 0.559188
- link LShoulder: mass 0.43527 -> 0.541429
- link LShoulderYaw_link: mass 0.69262 -> 0.861545
- link LThigh: mass 4.34097 -> 4.71096
- link LTibia: mass 2.50906 -> 2.72291
- link LWristRoll_link: mass 0.17551 -> 0.218316
- link LWristYaw_link: mass 0.061 -> 0.0758774
- link NeckPitch_link: mass 0.29923 -> 0.345282
- link NeckYaw_link: mass 0.32745 -> 0.377845
- link RAnklePitch_link: mass 0.42803 -> 0.464512
- link RElbow: mass 0.36997 -> 0.460203
- link RForeArm: mass 0.48271 -> 0.600439
- link RHip: mass 0.65864 -> 0.714778
- link RHipYaw_link: mass 0.51527 -> 0.559188
- link RShoulder: mass 0.43527 -> 0.541429
- link RShoulderYaw_link: mass 0.69262 -> 0.861545
- link RThigh: mass 4.34097 -> 4.71096
- link RTibia: mass 2.50906 -> 2.72291
- link RWristRoll_link: mass 0.17551 -> 0.218316
- link RWristYaw_link: mass 0.061 -> 0.0758774
- link body: mass 4.4142 -> 5.11337
- link l_ankle: mass 0.98379 -> 1.06764
- link l_wrist: mass 0.35549 -> 0.442191
- link r_ankle: mass 0.98379 -> 1.06764
- link r_wrist: mass 0.35549 -> 0.442191
- link torso: mass 5.0541 -> 5.85463

File: romeo_description/urdf/romeo_generated_urdf/romeo_arms.xacro (robot description, xacro)
@@ -13,6 +13,6 @@
 	<link name="LShoulder">
 		<inertial>
-			<mass value="0.43527"/>
-			<inertia ixx="0.000268738" ixy="-7.98278e-05" ixz="8.02495e-06" iyy="0.000151197" iyz="1.72313e-05" izz="0.000290161"/>
+			<mass value="0.541429"/>
+			<inertia ixx="0.00033428" ixy="-9.92972e-05" ixz="9.98217e-06" iyy="0.000188073" iyz="2.14339e-05" izz="0.000360929"/>
 			<origin rpy="0 0 0" xyz="-0.0112798 -0.0260712 0.00468882"/>
 		</inertial>
@@ -27,6 +27,6 @@
 	<link name="LShoulderYaw_link">
 		<inertial>
-			<mass value="0.69262"/>
-			<inertia ixx="0.000953111" ixy="0.000479248" ixz="0.000898232" iyy="0.00250956" iyz="-1.65544e-05" izz="0.00233103"/>
+			<mass value="0.861545"/>
+			<inertia ixx="0.00118557" ixy="0.000596133" ixz="0.0011173" iyy="0.00312162" iyz="-2.05919e-05" izz="0.00289955"/>
 			<origin rpy="0 0 0" xyz="0.0965281 0.00465308 0.00168775"/>
 		</inertial>
@@ -42,6 +42,6 @@
 	<link name="LForeArm">
 		<inertial>
-			<mass value="0.48271"/>
-			<inertia ixx="0.000166894" ixy="9.68978e-06" ixz="-1.49781e-05" iyy="0.000408141" iyz="1.2555e-06" izz="0.00036684"/>
+			<mass value="0.600439"/>
+			<inertia ixx="0.000207598" ixy="1.2053e-05" ixz="-1.86312e-05" iyy="0.000507683" iyz="1.56171e-06" izz="0.000456309"/>
 			<origin rpy="0 0 0" xyz="-0.0348859 -0.0011589 -0.00148134"/>
 		</inertial>
@@ -56,6 +56,6 @@
 	<link name="LElbow">
 		<inertial>
-			<mass value="0.36997"/>
-			<inertia ixx="0.000404839" ixy="0.000470943" ixz="2.57237e-05" iyy="0.00102723" iyz="2.9528e-05" izz="0.000987329"/>
+			<mass value="0.460203"/>
+			<inertia ixx="0.000503576" ixy="0.000585803" ixz="3.19975e-05" iyy="0.00127777" iyz="3.67296e-05" izz="0.00122813"/>
 			<origin rpy="0 0 0" xyz="0.068523 0.0097 0.00458766"/>
 		</inertial>
@@ -71,6 +71,6 @@
 	<link name="LWristRoll_link">
 		<inertial>
-			<mass value="0.17551"/>
-			<inertia ixx="8.1046e-05" ixy="-1.46219e-06" ixz="-3.67139e-05" iyy="0.000308979" iyz="-8.92509e-08" izz="0.000294305"/>
+			<mass value="0.218316"/>
+			<inertia ixx="0.000100812" ixy="-1.81881e-06" ixz="-4.56681e-05" iyy="0.000384336" iyz="-1.11019e-07" izz="0.000366084"/>
 			<origin rpy="0 0 0" xyz="-0.0592449 6e-05 -0.00144745"/>
 		</inertial>
@@ -86,6 +86,6 @@
 	<link name="LWristYaw_link">
 		<inertial>
-			<mass value="0.061"/>
-			<inertia ixx="1.25161e-05" ixy="-4.16668e-08" ixz="-7.01768e-07" iyy="2.83374e-05" iyz="1.56375e-08" izz="2.79694e-05"/>
+			<mass value="0.0758774"/>
+			<inertia ixx="1.55687e-05" ixy="-5.1829e-08" ixz="-8.72923e-07" iyy="3.52487e-05" iyz="1.94513e-08" izz="3.4791e-05"/>
 			<origin rpy="0 0 0" xyz="-0.00657144 0.00017 -0.000115829"/>
 		</inertial>
@@ -101,6 +101,6 @@
 	<link name="l_wrist">
 		<inertial>
-			<mass value="0.35549"/>
-			<inertia ixx="0.000325271" ixy="-0.000324985" ixz="1.52493e-05" iyy="0.000666741" iyz="6.27901e-05" izz="0.000820118"/>
+			<mass value="0.442191"/>
+			<inertia ixx="0.000404603" ixy="-0.000404247" ixz="1.89685e-05" iyy="0.000829354" iyz="7.81042e-05" izz="0.00102014"/>
 			<origin rpy="0 0 0" xyz="0.07358 -0.00628 -0.00098"/>
 		</inertial>
@@ -129,6 +129,6 @@
 	<link name="RShoulder">
 		<inertial>
-			<mass value="0.43527"/>
-			<inertia ixx="0.000264235" ixy="8.24341e-05" ixz="1.55448e-05" iyy="0.000160752" iyz="-3.06968e-05" izz="0.000285109"/>
+			<mass value="0.541429"/>
+			<inertia ixx="0.00032868" ixy="0.000102539" ixz="1.9336e-05" iyy="0.000199958" iyz="-3.81835e-05" izz="0.000354645"/>
 			<origin rpy="0 0 0" xyz="-0.0112798 0.0260712 0.00468882"/>
 		</inertial>
@@ -143,6 +143,6 @@
 	<link name="RShoulderYaw_link">
 		<inertial>
-			<mass value="0.69262"/>
-			<inertia ixx="0.000955527" ixy="-0.000291705" ixz="0.000927729" iyy="0.00250758" iyz="1.49948e-05" izz="0.00233059"/>
+			<mass value="0.861545"/>
+			<inertia ixx="0.00118857" ixy="-0.00036285" ixz="0.001154" iyy="0.00311916" iyz="1.86519e-05" izz="0.002899"/>
 			<origin rpy="0 0 0" xyz="0.0965281 -0.00465308 0.00168775"/>
 		</inertial>
@@ -158,6 +158,6 @@
 	<link name="RForeArm">
 		<inertial>
-			<mass value="0.48271"/>
-			<inertia ixx="0.000166993" ixy="-6.12728e-06" ixz="-1.49476e-05" iyy="0.000408038" iyz="7.67117e-07" izz="0.000366843"/>
+			<mass value="0.600439"/>
+			<inertia ixx="0.000207722" ixy="-7.62167e-06" ixz="-1.85932e-05" iyy="0.000507556" iyz="9.54211e-07" izz="0.000456313"/>
 			<origin rpy="0 0 0" xyz="-0.0348859 0.0011589 -0.00148134"/>
 		</inertial>
@@ -172,6 +172,6 @@
 	<link name="RElbow">
 		<inertial>
-			<mass value="0.36997"/>
-			<inertia ixx="0.000404839" ixy="-2.08748e-05" ixz="2.57237e-05" iyy="0.00102723" iyz="-3.39957e-06" izz="0.000987329"/>
+			<mass value="0.460203"/>
+			<inertia ixx="0.000503576" ixy="-2.59661e-05" ixz="3.19975e-05" iyy="0.00127777" iyz="-4.2287e-06" izz="0.00122813"/>
 			<origin rpy="0 0 0" xyz="0.068523 -0.0097 0.00458766"/>
 		</inertial>
@@ -187,6 +187,6 @@
 	<link name="RWristRoll_link">
 		<inertial>
-			<mass value="0.17551"/>
-			<inertia ixx="8.1046e-05" ixy="-2.14425e-07" ixz="-3.67139e-05" iyy="0.000308979" iyz="-5.87658e-08" izz="0.000294305"/>
+			<mass value="0.218316"/>
+			<inertia ixx="0.000100812" ixy="-2.66721e-07" ixz="-4.56681e-05" iyy="0.000384336" iyz="-7.30984e-08" izz="0.000366084"/>
 			<origin rpy="0 0 0" xyz="-0.0592449 -6e-05 -0.00144745"/>
 		</inertial>
@@ -202,6 +202,6 @@
 	<link name="RWristYaw_link">
 		<inertial>
-			<mass value="0.061"/>
-			<inertia ixx="1.25161e-05" ixy="9.4625e-08" ixz="-7.01768e-07" iyy="2.83374e-05" iyz="1.80397e-08" izz="2.79694e-05"/>
+			<mass value="0.0758774"/>
+			<inertia ixx="1.55687e-05" ixy="1.17703e-07" ixz="-8.72923e-07" iyy="3.52487e-05" iyz="2.24395e-08" izz="3.4791e-05"/>
 			<origin rpy="0 0 0" xyz="-0.00657144 -0.00017 -0.000115829"/>
 		</inertial>
@@ -217,6 +217,6 @@
 	<link name="r_wrist">
 		<inertial>
-			<mass value="0.35549"/>
-			<inertia ixx="0.000325271" ixy="3.54589e-06" ixz="1.52493e-05" iyy="0.000666741" iyz="5.84145e-05" izz="0.000820118"/>
+			<mass value="0.442191"/>
+			<inertia ixx="0.000404603" ixy="4.4107e-06" ixz="1.89685e-05" iyy="0.000829354" iyz="7.26613e-05" izz="0.00102014"/>
 			<origin rpy="0 0 0" xyz="0.07358 0.00628 -0.00098"/>
 		</inertial>

File: romeo_description/urdf/romeo_generated_urdf/romeo_fingers.xacro (robot description, xacro)
@@ -3,5 +3,5 @@
  ****** File automatically generated by generate_urdf.py script ******
  *********************************************************************-->
-<robot name="romeoH37" xmlns:xacro="http://www.ros.org/wiki/xacro">
+<robot name="RomeoH37" xmlns:xacro="http://www.ros.org/wiki/xacro">
 	<link name="RFinger13_link">
 		<inertial>

File: romeo_description/urdf/romeo_generated_urdf/romeo_head.xacro (robot description, xacro)
@@ -13,6 +13,6 @@
 	<link name="NeckYaw_link">
 		<inertial>
-			<mass value="0.32745"/>
-			<inertia ixx="0.000242012" ixy="-2.69441e-07" ixz="-1.29328e-05" iyy="0.000225485" iyz="-6.99834e-07" izz="7.29248e-05"/>
+			<mass value="0.377845"/>
+			<inertia ixx="0.000279258" ixy="-3.10908e-07" ixz="-1.49231e-05" iyy="0.000260188" iyz="-8.07538e-07" izz="8.41479e-05"/>
 			<origin rpy="0 0 0" xyz="-0.00635646 0 -0.030002"/>
 		</inertial>
@@ -27,6 +27,6 @@
 	<link name="NeckPitch_link">
 		<inertial>
-			<mass value="0.29923"/>
-			<inertia ixx="0.000412832" ixy="-1.67846e-06" ixz="0.000111721" iyy="0.000383921" iyz="5.04259e-05" izz="0.000264006"/>
+			<mass value="0.345282"/>
+			<inertia ixx="0.000476367" ixy="-1.93678e-06" ixz="0.000128915" iyy="0.000443007" iyz="5.81865e-05" izz="0.000304636"/>
 			<origin rpy="0 0 0" xyz="0.00372 0 0.04811"/>
 		</inertial>
@@ -42,6 +42,6 @@
 	<link name="HeadPitch_link">
 		<inertial>
-			<mass value="0.13728"/>
-			<inertia ixx="2.23022e-05" ixy="1.3103e-07" ixz="-1.31933e-05" iyy="6.44652e-05" iyz="-4.26e-09" izz="5.78637e-05"/>
+			<mass value="0.158407"/>
+			<inertia ixx="2.57346e-05" ixy="1.51196e-07" ixz="-1.52238e-05" iyy="7.43865e-05" iyz="-4.91562e-09" izz="6.6769e-05"/>
 			<origin rpy="0 0 0" xyz="0.0014 0 -0.00462"/>
 		</inertial>
@@ -56,6 +56,6 @@
 	<link name="HeadRoll_link">
 		<inertial>
-			<mass value="1.79432"/>
-			<inertia ixx="0.00808695" ixy="-3.36239e-05" ixz="0.00239535" iyy="0.00960886" iyz="0.000260292" izz="0.00796332"/>
+			<mass value="2.07047"/>
+			<inertia ixx="0.00933153" ixy="-3.87986e-05" ixz="0.002764" iyy="0.0110877" iyz="0.000300351" izz="0.00918888"/>
 			<origin rpy="0 0 0" xyz="0.01263 0 0.07498"/>
 		</inertial>

File: romeo_description/urdf/romeo_generated_urdf/romeo_legs.xacro (robot description, xacro)
@@ -13,6 +13,6 @@
 	<link name="LHipYaw_link">
 		<inertial>
-			<mass value="0.51527"/>
-			<inertia ixx="0.000797373" ixy="-1.0184e-06" ixz="-0.000231697" iyy="0.00131776" iyz="3.91707e-06" izz="0.000785018"/>
+			<mass value="0.559188"/>
+			<inertia ixx="0.000865336" ixy="-1.1052e-06" ixz="-0.000251445" iyy="0.00143007" iyz="4.25093e-06" izz="0.000851928"/>
 			<origin rpy="0 0 0" xyz="-0.00922 -0.00167 0.042"/>
 		</inertial>
@@ -27,6 +27,6 @@
 	<link name="LHip">
 		<inertial>
-			<mass value="0.65864"/>
-			<inertia ixx="0.000863659" ixy="-6.20354e-06" ixz="-1.86793e-06" iyy="0.000505068" iyz="1.24373e-06" izz="0.000938555"/>
+			<mass value="0.714778"/>
+			<inertia ixx="0.000937272" ixy="-6.73228e-06" ixz="-2.02714e-06" iyy="0.000548117" iyz="1.34974e-06" izz="0.00101855"/>
 			<origin rpy="0 0 0" xyz="0.00249 -0.00205 -0.00147"/>
 		</inertial>
@@ -41,6 +41,6 @@
 	<link name="LThigh">
 		<inertial>
-			<mass value="4.34097"/>
-			<inertia ixx="0.036002" ixy="-2.22796e-05" ixz="0.0230461" iyy="0.0364084" iyz="0.00065633" izz="0.0112971"/>
+			<mass value="4.71096"/>
+			<inertia ixx="0.0390706" ixy="-2.41786e-05" ixz="0.0250104" iyy="0.0395116" iyz="0.000712271" izz="0.0122599"/>
 			<origin rpy="0 0 0" xyz="-0.02138 -0.00255 -0.14577"/>
 		</inertial>
@@ -56,6 +56,6 @@
 	<link name="LTibia">
 		<inertial>
-			<mass value="2.50906"/>
-			<inertia ixx="0.0146626" ixy="5.06229e-08" ixz="0.00278247" iyy="0.0145661" iyz="-5.66452e-06" izz="0.00340234"/>
+			<mass value="2.72291"/>
+			<inertia ixx="0.0159124" ixy="5.49385e-08" ixz="0.00301963" iyy="0.0158076" iyz="-6.1473e-06" izz="0.00369233"/>
 			<origin rpy="0 0 0" xyz="-0.00415 -0.00054 -0.11011"/>
 		</inertial>
@@ -71,6 +71,6 @@
 	<link name="LAnklePitch_link">
 		<inertial>
-			<mass value="0.42803"/>
-			<inertia ixx="0.000338486" ixy="-1.0818e-07" ixz="9.621e-08" iyy="0.000220504" iyz="-1.13514e-06" izz="0.00039211"/>
+			<mass value="0.464512"/>
+			<inertia ixx="0.000367336" ixy="-1.174e-07" ixz="1.0441e-07" iyy="0.000239298" iyz="-1.23189e-06" izz="0.000425531"/>
 			<origin rpy="0 0 0" xyz="0.00132 -0.00117 0.00015"/>
 		</inertial>
@@ -85,6 +85,6 @@
 	<link name="l_ankle">
 		<inertial>
-			<mass value="0.98379"/>
-			<inertia ixx="0.000901343" ixy="-4.5809e-05" ixz="-0.000810091" iyy="0.00540559" iyz="5.65123e-05" izz="0.00543292"/>
+			<mass value="1.06764"/>
+			<inertia ixx="0.000978167" ixy="-4.97135e-05" ixz="-0.000879138" iyy="0.00586633" iyz="6.13291e-05" izz="0.00589599"/>
 			<origin rpy="0 0 0" xyz="0.0483878 0.00120158 -0.0367645"/>
 		</inertial>
@@ -107,6 +107,6 @@
 	<link name="RHipYaw_link">
 		<inertial>
-			<mass value="0.51527"/>
-			<inertia ixx="0.000797373" ixy="-1.6886e-05" ixz="-0.000231697" iyy="0.00131776" iyz="7.61991e-05" izz="0.000785018"/>
+			<mass value="0.559188"/>
+			<inertia ixx="0.000865336" ixy="-1.83253e-05" ixz="-0.000251445" iyy="0.00143007" iyz="8.26938e-05" izz="0.000851928"/>
 			<origin rpy="0 0 0" xyz="-0.00922 0.00167 0.042"/>
 		</inertial>
@@ -121,6 +121,6 @@
 	<link name="RHip">
 		<inertial>
-			<mass value="0.65864"/>
-			<inertia ixx="0.000863659" ixy="5.20518e-07" ixz="-1.86793e-06" iyy="0.000505068" iyz="-2.72589e-06" izz="0.000938555"/>
+			<mass value="0.714778"/>
+			<inertia ixx="0.000937272" ixy="5.64884e-07" ixz="-2.02714e-06" iyy="0.000548117" iyz="-2.95823e-06" izz="0.00101855"/>
 			<origin rpy="0 0 0" xyz="0.00249 0.00205 -0.00147"/>
 		</inertial>
@@ -135,6 +135,6 @@
 	<link name="RThigh">
 		<inertial>
-			<mass value="4.34097"/>
-			<inertia ixx="0.036002" ixy="-0.00049561" ixz="0.0230461" iyy="0.0364084" iyz="-0.00257086" izz="0.0112971"/>
+			<mass value="4.71096"/>
+			<inertia ixx="0.0390706" ixy="-0.000537853" ixz="0.0250104" iyy="0.0395116" iyz="-0.00278999" izz="0.0122599"/>
 			<origin rpy="0 0 0" xyz="-0.02138 0.00255 -0.14577"/>
 		</inertial>
@@ -150,6 +150,6 @@
 	<link name="RTibia">
 		<inertial>
-			<mass value="2.50906"/>
-			<inertia ixx="0.0146626" ixy="-1.1195e-05" ixz="0.00278247" iyy="0.0145661" iyz="-0.000304039" izz="0.00340234"/>
+			<mass value="2.72291"/>
+			<inertia ixx="0.0159124" ixy="-1.21492e-05" ixz="0.00301963" iyy="0.0158076" iyz="-0.000329953" izz="0.00369233"/>
 			<origin rpy="0 0 0" xyz="-0.00415 0.00054 -0.11011"/>
 		</inertial>
@@ -165,6 +165,6 @@
 	<link name="RAnklePitch_link">
 		<inertial>
-			<mass value="0.42803"/>
-			<inertia ixx="0.000338486" ixy="1.21392e-06" ixz="9.621e-08" iyy="0.000220504" iyz="-9.84901e-07" izz="0.00039211"/>
+			<mass value="0.464512"/>
+			<inertia ixx="0.000367336" ixy="1.31739e-06" ixz="1.0441e-07" iyy="0.000239298" iyz="-1.06885e-06" izz="0.000425531"/>
 			<origin rpy="0 0 0" xyz="0.00132 0.00117 0.00015"/>
 		</inertial>
@@ -179,6 +179,6 @@
 	<link name="r_ankle">
 		<inertial>
-			<mass value="0.98379"/>
-			<inertia ixx="0.000901343" ixy="-0.000160208" ixz="-0.000810091" iyy="0.00540559" iyz="0.000143431" izz="0.00543292"/>
+			<mass value="1.06764"/>
+			<inertia ixx="0.000978167" ixy="-0.000173863" ixz="-0.000879138" iyy="0.00586633" iyz="0.000155656" izz="0.00589599"/>
 			<origin rpy="0 0 0" xyz="0.0483878 -0.00120158 -0.0367645"/>
 		</inertial>

File: romeo_description/urdf/romeo_generated_urdf/romeo_robot.xacro (robot description, xacro)
@@ -3,5 +3,5 @@
  ****** File automatically generated by generate_urdf.py script ******
  *********************************************************************-->
-<robot name="romeoH37" xmlns:xacro="http://www.ros.org/wiki/xacro">
+<robot name="RomeoH37" xmlns:xacro="http://www.ros.org/wiki/xacro">
 	<xacro:include filename="romeo_visual_collisions.xacro"/>
 	<xacro:include filename="romeo_head.xacro"/>

File: romeo_description/urdf/romeo_generated_urdf/romeo_sensors.xacro (robot description, xacro)
@@ -3,5 +3,5 @@
  ****** File automatically generated by generate_urdf.py script ******
  *********************************************************************-->
-<robot name="romeoH37" xmlns:xacro="http://www.ros.org/wiki/xacro">
+<robot name="RomeoH37" xmlns:xacro="http://www.ros.org/wiki/xacro">
 	<link name="RFsrFToeRearRight_frame"/>
 	<joint name="RFoot/FSR/ToeRearRight_sensor_fixedjoint" type="fixed">

File: romeo_description/urdf/romeo_generated_urdf/romeo_torso.xacro (robot description, xacro)
@@ -13,6 +13,6 @@
 	<link name="torso">
 		<inertial>
-			<mass value="5.0541"/>
-			<inertia ixx="0.0623514" ixy="-3.02711e-06" ixz="0.0093264" iyy="0.0365041" iyz="-0.000132541" izz="0.0639535"/>
+			<mass value="5.85463"/>
+			<inertia ixx="0.0587116" ixy="-3.02711e-06" ixz="0.0101426" iyy="0.0326812" iyz="-0.000132541" izz="0.0637705"/>
 			<origin rpy="0 0 0" xyz="0.01512 0 0.06743"/>
 		</inertial>
@@ -28,6 +28,6 @@
 	<link name="body">
 		<inertial>
-			<mass value="4.4142"/>
-			<inertia ixx="0.0487058" ixy="6.27009e-05" ixz="-0.0496477" iyy="0.0449798" iyz="-2.92721e-05" izz="0.0182883"/>
+			<mass value="5.11337"/>
+			<inertia ixx="0.0564204" ixy="7.26322e-05" ixz="-0.0575115" iyy="0.0521042" iyz="-3.39086e-05" izz="0.021185"/>
 			<origin rpy="0 0 0" xyz="0.02825 0 -0.16653"/>
 		</inertial>
