Commit message: update to the latest Romeo URDF

File: romeo_description/urdf/romeo_generated_urdf/romeo_visual_collisions.xacro (robot description, xacro)
@@ -46,4 +46,480 @@
 		</collision>
 	</xacro:macro>
+	<xacro:macro name="insert_visu_RFinger12_link">
+		<visual>
+			<geometry>
+				<mesh filename="package://romeo_description/meshes/RFinger12.dae" scale="1 1 1"/>
+			</geometry>
+			<origin rpy="0 0 0" xyz="0 0 0"/>
+		</visual>
+		<collision>
+			<geometry>
+				<mesh filename="package://romeo_description/meshes/RFinger12_0.10.stl" scale="1 1 1"/>
+			</geometry>
+			<origin rpy="0 0 0" xyz="0 0 0"/>
+		</collision>
+	</xacro:macro>
+	<xacro:macro name="insert_visu_LFinger33_link">
+		<visual>
+			<geometry>
+				<mesh filename="package://romeo_description/meshes/LFinger33.dae" scale="1 1 1"/>
+			</geometry>
+			<origin rpy="0 0 0" xyz="0 0 0"/>
+		</visual>
+		<collision>
+			<geometry>
+				<mesh filename="package://romeo_description/meshes/LFinger33_0.10.stl" scale="1 1 1"/>
+			</geometry>
+			<origin rpy="0 0 0" xyz="0 0 0"/>
+		</collision>
+	</xacro:macro>
+	<xacro:macro name="insert_visu_RFinger31_link">
+		<visual>
+			<geometry>
+				<mesh filename="package://romeo_description/meshes/RFinger31.dae" scale="1 1 1"/>
+			</geometry>
+			<origin rpy="0 0 0" xyz="0 0 0"/>
+		</visual>
+		<collision>
+			<geometry>
+				<mesh filename="package://romeo_description/meshes/RFinger31_0.10.stl" scale="1 1 1"/>
+			</geometry>
+			<origin rpy="0 0 0" xyz="0 0 0"/>
+		</collision>
+	</xacro:macro>
+	<xacro:macro name="insert_visu_LWristYaw_link">
+		<visual>
+			<geometry>
+				<mesh filename="package://romeo_description/meshes/LWristYaw.dae" scale="1 1 1"/>
+			</geometry>
+			<origin rpy="0 0 0" xyz="0 0 0"/>
+		</visual>
+		<collision>
+			<geometry>
+				<mesh filename="package://romeo_description/meshes/LWristYaw_0.10.stl" scale="1 1 1"/>
+			</geometry>
+			<origin rpy="0 0 0" xyz="0 0 0"/>
+		</collision>
+	</xacro:macro>
+	<xacro:macro name="insert_visu_RFinger32_link">
+		<visual>
+			<geometry>
+				<mesh filename="package://romeo_description/meshes/RFinger32.dae" scale="1 1 1"/>
+			</geometry>
+			<origin rpy="0 0 0" xyz="0 0 0"/>
+		</visual>
+		<collision>
+			<geometry>
+				<mesh filename="package://romeo_description/meshes/RFinger32_0.10.stl" scale="1 1 1"/>
+			</geometry>
+			<origin rpy="0 0 0" xyz="0 0 0"/>
+		</collision>
+	</xacro:macro>
+	<xacro:macro name="insert_visu_LFinger21_link">
+		<visual>
+			<geometry>
+				<mesh filename="package://romeo_description/meshes/LFinger21.dae" scale="1 1 1"/>
+			</geometry>
+			<origin rpy="0 0 0" xyz="0 0 0"/>
+		</visual>
+		<collision>
+			<geometry>
+				<mesh filename="package://romeo_description/meshes/LFinger21_0.10.stl" scale="1 1 1"/>
+			</geometry>
+			<origin rpy="0 0 0" xyz="0 0 0"/>
+		</collision>
+	</xacro:macro>
+	<xacro:macro name="insert_visu_LFinger13_link">
+		<visual>
+			<geometry>
+				<mesh filename="package://romeo_description/meshes/LFinger13.dae" scale="1 1 1"/>
+			</geometry>
+			<origin rpy="0 0 0" xyz="0 0 0"/>
+		</visual>
+		<collision>
+			<geometry>
+				<mesh filename="package://romeo_description/meshes/LFinger13_0.10.stl" scale="1 1 1"/>
+			</geometry>
+			<origin rpy="0 0 0" xyz="0 0 0"/>
+		</collision>
+	</xacro:macro>
+	<xacro:macro name="insert_visu_LFinger32_link">
+		<visual>
+			<geometry>
+				<mesh filename="package://romeo_description/meshes/LFinger32.dae" scale="1 1 1"/>
+			</geometry>
+			<origin rpy="0 0 0" xyz="0 0 0"/>
+		</visual>
+		<collision>
+			<geometry>
+				<mesh filename="package://romeo_description/meshes/LFinger32_0.10.stl" scale="1 1 1"/>
+			</geometry>
+			<origin rpy="0 0 0" xyz="0 0 0"/>
+		</collision>
+	</xacro:macro>
+	<xacro:macro name="insert_visu_LThumb3_link">
+		<visual>
+			<geometry>
+				<mesh filename="package://romeo_description/meshes/LThumb3.dae" scale="1 1 1"/>
+			</geometry>
+			<origin rpy="0 0 0" xyz="0 0 0"/>
+		</visual>
+		<collision>
+			<geometry>
+				<mesh filename="package://romeo_description/meshes/LThumb3_0.10.stl" scale="1 1 1"/>
+			</geometry>
+			<origin rpy="0 0 0" xyz="0 0 0"/>
+		</collision>
+	</xacro:macro>
+	<xacro:macro name="insert_visu_HeadRoll_link">
+		<visual>
+			<geometry>
+				<mesh filename="package://romeo_description/meshes/HeadRoll.dae" scale="1 1 1"/>
+			</geometry>
+			<origin rpy="0 0 0" xyz="0 0 0"/>
+		</visual>
+		<collision>
+			<geometry>
+				<mesh filename="package://romeo_description/meshes/HeadRoll_0.10.stl" scale="1 1 1"/>
+			</geometry>
+			<origin rpy="0 0 0" xyz="0 0 0"/>
+		</collision>
+	</xacro:macro>
+	<xacro:macro name="insert_visu_LThumb1_link">
+		<visual>
+			<geometry>
+				<mesh filename="package://romeo_description/meshes/LThumb1.dae" scale="1 1 1"/>
+			</geometry>
+			<origin rpy="0 0 0" xyz="0 0 0"/>
+		</visual>
+		<collision>
+			<geometry>
+				<mesh filename="package://romeo_description/meshes/LThumb1_0.10.stl" scale="1 1 1"/>
+			</geometry>
+			<origin rpy="0 0 0" xyz="0 0 0"/>
+		</collision>
+	</xacro:macro>
+	<xacro:macro name="insert_visu_LFinger11_link">
+		<visual>
+			<geometry>
+				<mesh filename="package://romeo_description/meshes/LFinger11.dae" scale="1 1 1"/>
+			</geometry>
+			<origin rpy="0 0 0" xyz="0 0 0"/>
+		</visual>
+		<collision>
+			<geometry>
+				<mesh filename="package://romeo_description/meshes/LFinger11_0.10.stl" scale="1 1 1"/>
+			</geometry>
+			<origin rpy="0 0 0" xyz="0 0 0"/>
+		</collision>
+	</xacro:macro>
+	<xacro:macro name="insert_visu_RFinger22_link">
+		<visual>
+			<geometry>
+				<mesh filename="package://romeo_description/meshes/RFinger22.dae" scale="1 1 1"/>
+			</geometry>
+			<origin rpy="0 0 0" xyz="0 0 0"/>
+		</visual>
+		<collision>
+			<geometry>
+				<mesh filename="package://romeo_description/meshes/RFinger22_0.10.stl" scale="1 1 1"/>
+			</geometry>
+			<origin rpy="0 0 0" xyz="0 0 0"/>
+		</collision>
+	</xacro:macro>
+	<xacro:macro name="insert_visu_LFinger22_link">
+		<visual>
+			<geometry>
+				<mesh filename="package://romeo_description/meshes/LFinger22.dae" scale="1 1 1"/>
+			</geometry>
+			<origin rpy="0 0 0" xyz="0 0 0"/>
+		</visual>
+		<collision>
+			<geometry>
+				<mesh filename="package://romeo_description/meshes/LFinger22_0.10.stl" scale="1 1 1"/>
+			</geometry>
+			<origin rpy="0 0 0" xyz="0 0 0"/>
+		</collision>
+	</xacro:macro>
+	<xacro:macro name="insert_visu_RFinger21_link">
+		<visual>
+			<geometry>
+				<mesh filename="package://romeo_description/meshes/RFinger21.dae" scale="1 1 1"/>
+			</geometry>
+			<origin rpy="0 0 0" xyz="0 0 0"/>
+		</visual>
+		<collision>
+			<geometry>
+				<mesh filename="package://romeo_description/meshes/RFinger21_0.10.stl" scale="1 1 1"/>
+			</geometry>
+			<origin rpy="0 0 0" xyz="0 0 0"/>
+		</collision>
+	</xacro:macro>
+	<xacro:macro name="insert_visu_RShoulderYaw_link">
+		<visual>
+			<geometry>
+				<mesh filename="package://romeo_description/meshes/RShoulderYaw.dae" scale="1 1 1"/>
+			</geometry>
+			<origin rpy="0 0 0" xyz="0 0 0"/>
+		</visual>
+		<collision>
+			<geometry>
+				<mesh filename="package://romeo_description/meshes/RShoulderYaw_0.10.stl" scale="1 1 1"/>
+			</geometry>
+			<origin rpy="0 0 0" xyz="0 0 0"/>
+		</collision>
+	</xacro:macro>
+	<xacro:macro name="insert_visu_LWristRoll_link">
+		<visual>
+			<geometry>
+				<mesh filename="package://romeo_description/meshes/LWristRoll.dae" scale="1 1 1"/>
+			</geometry>
+			<origin rpy="0 0 0" xyz="0 0 0"/>
+		</visual>
+		<collision>
+			<geometry>
+				<mesh filename="package://romeo_description/meshes/LWristRoll_0.10.stl" scale="1 1 1"/>
+			</geometry>
+			<origin rpy="0 0 0" xyz="0 0 0"/>
+		</collision>
+	</xacro:macro>
+	<xacro:macro name="insert_visu_RThumb1_link">
+		<visual>
+			<geometry>
+				<mesh filename="package://romeo_description/meshes/RThumb1.dae" scale="1 1 1"/>
+			</geometry>
+			<origin rpy="0 0 0" xyz="0 0 0"/>
+		</visual>
+		<collision>
+			<geometry>
+				<mesh filename="package://romeo_description/meshes/RThumb1_0.10.stl" scale="1 1 1"/>
+			</geometry>
+			<origin rpy="0 0 0" xyz="0 0 0"/>
+		</collision>
+	</xacro:macro>
+	<xacro:macro name="insert_visu_body">
+		<visual>
+			<geometry>
+				<mesh filename="package://romeo_description/meshes/TrunkYaw.dae" scale="1 1 1"/>
+			</geometry>
+			<origin rpy="0 0 0" xyz="0 0 0"/>
+		</visual>
+		<collision>
+			<geometry>
+				<mesh filename="package://romeo_description/meshes/TrunkYaw_0.10.stl" scale="1 1 1"/>
+			</geometry>
+			<origin rpy="0 0 0" xyz="0 0 0"/>
+		</collision>
+	</xacro:macro>
+	<xacro:macro name="insert_visu_RThumb2_link">
+		<visual>
+			<geometry>
+				<mesh filename="package://romeo_description/meshes/RThumb2.dae" scale="1 1 1"/>
+			</geometry>
+			<origin rpy="0 0 0" xyz="0 0 0"/>
+		</visual>
+		<collision>
+			<geometry>
+				<mesh filename="package://romeo_description/meshes/RThumb2_0.10.stl" scale="1 1 1"/>
+			</geometry>
+			<origin rpy="0 0 0" xyz="0 0 0"/>
+		</collision>
+	</xacro:macro>
+	<xacro:macro name="insert_visu_r_wrist">
+		<visual>
+			<geometry>
+				<mesh filename="package://romeo_description/meshes/RWristPitch.dae" scale="1 1 1"/>
+			</geometry>
+			<origin rpy="0 0 0" xyz="0 0 0"/>
+		</visual>
+		<collision>
+			<geometry>
+				<mesh filename="package://romeo_description/meshes/RWristPitch_0.10.stl" scale="1 1 1"/>
+			</geometry>
+			<origin rpy="0 0 0" xyz="0 0 0"/>
+		</collision>
+	</xacro:macro>
+	<xacro:macro name="insert_visu_NeckPitch_link">
+		<visual>
+			<geometry>
+				<mesh filename="package://romeo_description/meshes/NeckPitch.dae" scale="1 1 1"/>
+			</geometry>
+			<origin rpy="0 0 0" xyz="0 0 0"/>
+		</visual>
+		<collision>
+			<geometry>
+				<mesh filename="package://romeo_description/meshes/NeckPitch_0.10.stl" scale="1 1 1"/>
+			</geometry>
+			<origin rpy="0 0 0" xyz="0 0 0"/>
+		</collision>
+	</xacro:macro>
+	<xacro:macro name="insert_visu_LThumb2_link">
+		<visual>
+			<geometry>
+				<mesh filename="package://romeo_description/meshes/LThumb2.dae" scale="1 1 1"/>
+			</geometry>
+			<origin rpy="0 0 0" xyz="0 0 0"/>
+		</visual>
+		<collision>
+			<geometry>
+				<mesh filename="package://romeo_description/meshes/LThumb2_0.10.stl" scale="1 1 1"/>
+			</geometry>
+			<origin rpy="0 0 0" xyz="0 0 0"/>
+		</collision>
+	</xacro:macro>
+	<xacro:macro name="insert_visu_LFinger12_link">
+		<visual>
+			<geometry>
+				<mesh filename="package://romeo_description/meshes/LFinger12.dae" scale="1 1 1"/>
+			</geometry>
+			<origin rpy="0 0 0" xyz="0 0 0"/>
+		</visual>
+		<collision>
+			<geometry>
+				<mesh filename="package://romeo_description/meshes/LFinger12_0.10.stl" scale="1 1 1"/>
+			</geometry>
+			<origin rpy="0 0 0" xyz="0 0 0"/>
+		</collision>
+	</xacro:macro>
+	<xacro:macro name="insert_visu_RTibia">
+		<visual>
+			<geometry>
+				<mesh filename="package://romeo_description/meshes/RKneePitch.dae" scale="1 1 1"/>
+			</geometry>
+			<origin rpy="0 0 0" xyz="0 0 0"/>
+		</visual>
+		<collision>
+			<geometry>
+				<mesh filename="package://romeo_description/meshes/RKneePitch_0.10.stl" scale="1 1 1"/>
+			</geometry>
+			<origin rpy="0 0 0" xyz="0 0 0"/>
+		</collision>
+	</xacro:macro>
+	<xacro:macro name="insert_visu_LEye">
+		<visual>
+			<geometry>
+				<mesh filename="package://romeo_description/meshes/LEyePitch.dae" scale="1 1 1"/>
+			</geometry>
+			<origin rpy="0 0 0" xyz="0 0 0"/>
+		</visual>
+		<collision>
+			<geometry>
+				<mesh filename="package://romeo_description/meshes/LEyePitch_0.10.stl" scale="1 1 1"/>
+			</geometry>
+			<origin rpy="0 0 0" xyz="0 0 0"/>
+		</collision>
+	</xacro:macro>
+	<xacro:macro name="insert_visu_RWristRoll_link">
+		<visual>
+			<geometry>
+				<mesh filename="package://romeo_description/meshes/RWristRoll.dae" scale="1 1 1"/>
+			</geometry>
+			<origin rpy="0 0 0" xyz="0 0 0"/>
+		</visual>
+		<collision>
+			<geometry>
+				<mesh filename="package://romeo_description/meshes/RWristRoll_0.10.stl" scale="1 1 1"/>
+			</geometry>
+			<origin rpy="0 0 0" xyz="0 0 0"/>
+		</collision>
+	</xacro:macro>
+	<xacro:macro name="insert_visu_RFinger23_link">
+		<visual>
+			<geometry>
+				<mesh filename="package://romeo_description/meshes/RFinger23.dae" scale="1 1 1"/>
+			</geometry>
+			<origin rpy="0 0 0" xyz="0 0 0"/>
+		</visual>
+		<collision>
+			<geometry>
+				<mesh filename="package://romeo_description/meshes/RFinger23_0.10.stl" scale="1 1 1"/>
+			</geometry>
+			<origin rpy="0 0 0" xyz="0 0 0"/>
+		</collision>
+	</xacro:macro>
+	<xacro:macro name="insert_visu_LThigh">
+		<visual>
+			<geometry>
+				<mesh filename="package://romeo_description/meshes/LHipPitch.dae" scale="1 1 1"/>
+			</geometry>
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
Commit message: update to the latest naoqi_tools script

File: romeo_description/urdf/romeo_generated_urdf/romeo.urdf (robot description, URDF)
Before this commit: robot RomeoH37, 96 links, 95 joints
Links:
- link LFsrFToeFrontLeft_frame: mass None -> 2e-06; geometry collision box size=0.01 0.01 0.005
- link LFsrFToeFrontRight_frame: mass None -> 2e-06; geometry collision box size=0.01 0.01 0.005
- link LFsrFToeRearLeft_frame: mass None -> 2e-06; geometry collision box size=0.01 0.01 0.005
- link LFsrFToeRearRight_frame: mass None -> 2e-06; geometry collision box size=0.01 0.01 0.005
- link LFsrFrontCenter_frame: mass None -> 2e-06; geometry collision box size=0.01 0.01 0.005
- link LFsrHeelLeft_frame: mass None -> 2e-06; geometry collision box size=0.01 0.01 0.005
- link LFsrHeelRight_frame: mass None -> 2e-06; geometry collision box size=0.01 0.01 0.005
- link LFsrRearCenter_frame: mass None -> 2e-06; geometry collision box size=0.01 0.01 0.005
- link RFsrFToeFrontLeft_frame: mass None -> 2e-06; geometry collision box size=0.01 0.01 0.005
- link RFsrFToeFrontRight_frame: mass None -> 2e-06; geometry collision box size=0.01 0.01 0.005
- link RFsrFToeRearLeft_frame: mass None -> 2e-06; geometry collision box size=0.01 0.01 0.005
- link RFsrFToeRearRight_frame: mass None -> 2e-06; geometry collision box size=0.01 0.01 0.005
- link RFsrFrontCenter_frame: mass None -> 2e-06; geometry collision box size=0.01 0.01 0.005
- link RFsrHeelLeft_frame: mass None -> 2e-06; geometry collision box size=0.01 0.01 0.005
- link RFsrHeelRight_frame: mass None -> 2e-06; geometry collision box size=0.01 0.01 0.005
- link RFsrRearCenter_frame: mass None -> 2e-06; geometry collision box size=0.01 0.01 0.005

File: romeo_description/urdf/romeo_generated_urdf/romeo_sensors.xacro (robot description, xacro)
@@ -4,5 +4,16 @@
  *********************************************************************-->
 <robot name="RomeoH37" xmlns:xacro="http://www.ros.org/wiki/xacro">
-	<link name="RFsrFToeRearRight_frame"/>
+	<link name="RFsrFToeRearRight_frame">
+		<collision>
+			<geometry>
+				<box size="0.01 0.01 0.005"/>
+			</geometry>
+			<origin rpy="0 0 0" xyz="0 0 0"/>
+		</collision>
+		<inertial>
+			<mass value="2e-06"/>
+			<inertia ixx="1.1e-09" ixy="0" ixz="0" iyy="1.1e-09" iyz="0" izz="1.1e-09"/>
+		</inertial>
+	</link>
 	<joint name="RFoot/FSR/ToeRearRight_sensor_fixedjoint" type="fixed">
 		<parent link="r_ankle"/>
@@ -25,5 +36,16 @@
 		<axis xyz="0 0 0"/>
 	</joint>
-	<link name="RFsrRearCenter_frame"/>
+	<link name="RFsrRearCenter_frame">
+		<collision>
+			<geometry>
+				<box size="0.01 0.01 0.005"/>
+			</geometry>
+			<origin rpy="0 0 0" xyz="0 0 0"/>
+		</collision>
+		<inertial>
+			<mass value="2e-06"/>
+			<inertia ixx="1.1e-09" ixy="0" ixz="0" iyy="1.1e-09" iyz="0" izz="1.1e-09"/>
+		</inertial>
+	</link>
 	<joint name="RFoot/FSR/CenterRear_sensor_fixedjoint" type="fixed">
 		<parent link="r_ankle"/>
@@ -32,5 +54,16 @@
 		<axis xyz="0 0 0"/>
 	</joint>
-	<link name="RFsrFrontCenter_frame"/>
+	<link name="RFsrFrontCenter_frame">
+		<collision>
+			<geometry>
+				<box size="0.01 0.01 0.005"/>
+			</geometry>
+			<origin rpy="0 0 0" xyz="0 0 0"/>
+		</collision>
+		<inertial>
+			<mass value="2e-06"/>
+			<inertia ixx="1.1e-09" ixy="0" ixz="0" iyy="1.1e-09" iyz="0" izz="1.1e-09"/>
+		</inertial>
+	</link>
 	<joint name="RFoot/FSR/CenterFront_sensor_fixedjoint" type="fixed">
 		<parent link="r_ankle"/>
@@ -45,5 +78,16 @@
 		<origin rpy="-1.57079632679 0 -1.57079632679" xyz="0 0 0"/>
 	</joint>
-	<link name="LFsrHeelRight_frame"/>
+	<link name="LFsrHeelRight_frame">
+		<collision>
+			<geometry>
+				<box size="0.01 0.01 0.005"/>
+			</geometry>
+			<origin rpy="0 0 0" xyz="0 0 0"/>
+		</collision>
+		<inertial>
+			<mass value="2e-06"/>
+			<inertia ixx="1.1e-09" ixy="0" ixz="0" iyy="1.1e-09" iyz="0" izz="1.1e-09"/>
+		</inertial>
+	</link>
 	<joint name="LFoot/FSR/HeelRight_sensor_fixedjoint" type="fixed">
 		<parent link="l_ankle"/>
@@ -71,5 +115,16 @@
 		<origin rpy="-1.57079632679 0 -1.57079632679" xyz="0 0 0"/>
 	</joint>
-	<link name="RFsrFToeFrontRight_frame"/>
+	<link name="RFsrFToeFrontRight_frame">
+		<collision>
+			<geometry>
+				<box size="0.01 0.01 0.005"/>
+			</geometry>
+			<origin rpy="0 0 0" xyz="0 0 0"/>
+		</collision>
+		<inertial>
+			<mass value="2e-06"/>
+			<inertia ixx="1.1e-09" ixy="0" ixz="0" iyy="1.1e-09" iyz="0" izz="1.1e-09"/>
+		</inertial>
+	</link>
 	<joint name="RFoot/FSR/ToeFrontRight_sensor_fixedjoint" type="fixed">
 		<parent link="r_ankle"/>
@@ -78,5 +133,16 @@
 		<axis xyz="0 0 0"/>
 	</joint>
-	<link name="RFsrHeelRight_frame"/>
+	<link name="RFsrHeelRight_frame">
+		<collision>
+			<geometry>
+				<box size="0.01 0.01 0.005"/>
+			</geometry>
+			<origin rpy="0 0 0" xyz="0 0 0"/>
+		</collision>
+		<inertial>
+			<mass value="2e-06"/>
+			<inertia ixx="1.1e-09" ixy="0" ixz="0" iyy="1.1e-09" iyz="0" izz="1.1e-09"/>
+		</inertial>
+	</link>
 	<joint name="RFoot/FSR/HeelRight_sensor_fixedjoint" type="fixed">
 		<parent link="r_ankle"/>
@@ -85,5 +151,16 @@
 		<axis xyz="0 0 0"/>
 	</joint>
-	<link name="RFsrFToeRearLeft_frame"/>
+	<link name="RFsrFToeRearLeft_frame">
+		<collision>
+			<geometry>
+				<box size="0.01 0.01 0.005"/>
+			</geometry>
+			<origin rpy="0 0 0" xyz="0 0 0"/>
+		</collision>
+		<inertial>
+			<mass value="2e-06"/>
+			<inertia ixx="1.1e-09" ixy="0" ixz="0" iyy="1.1e-09" iyz="0" izz="1.1e-09"/>
+		</inertial>
+	</link>
 	<joint name="RFoot/FSR/ToeRearLeft_sensor_fixedjoint" type="fixed">
 		<parent link="r_ankle"/>
@@ -99,5 +176,16 @@
 		<axis xyz="0 0 0"/>
 	</joint>
-	<link name="LFsrFToeRearRight_frame"/>
+	<link name="LFsrFToeRearRight_frame">
+		<collision>
+			<geometry>
+				<box size="0.01 0.01 0.005"/>
+			</geometry>
+			<origin rpy="0 0 0" xyz="0 0 0"/>
+		</collision>
+		<inertial>
+			<mass value="2e-06"/>
+			<inertia ixx="1.1e-09" ixy="0" ixz="0" iyy="1.1e-09" iyz="0" izz="1.1e-09"/>
+		</inertial>
+	</link>
 	<joint name="LFoot/FSR/ToeRearRight_sensor_fixedjoint" type="fixed">
 		<parent link="l_ankle"/>
@@ -106,5 +194,16 @@
 		<axis xyz="0 0 0"/>
 	</joint>
-	<link name="LFsrHeelLeft_frame"/>
+	<link name="LFsrHeelLeft_frame">
+		<collision>
+			<geometry>
+				<box size="0.01 0.01 0.005"/>
+			</geometry>
+			<origin rpy="0 0 0" xyz="0 0 0"/>
+		</collision>
+		<inertial>
+			<mass value="2e-06"/>
+			<inertia ixx="1.1e-09" ixy="0" ixz="0" iyy="1.1e-09" iyz="0" izz="1.1e-09"/>
+		</inertial>
+	</link>
 	<joint name="LFoot/FSR/HeelLeft_sensor_fixedjoint" type="fixed">
 		<parent link="l_ankle"/>
@@ -127,5 +226,16 @@
 		<axis xyz="0 0 0"/>
 	</joint>
-	<link name="LFsrFToeRearLeft_frame"/>
+	<link name="LFsrFToeRearLeft_frame">
+		<collision>
+			<geometry>
+				<box size="0.01 0.01 0.005"/>
+			</geometry>
+			<origin rpy="0 0 0" xyz="0 0 0"/>
+		</collision>
+		<inertial>
+			<mass value="2e-06"/>
+			<inertia ixx="1.1e-09" ixy="0" ixz="0" iyy="1.1e-09" iyz="0" izz="1.1e-09"/>
+		</inertial>
+	</link>
 	<joint name="LFoot/FSR/ToeRearLeft_sensor_fixedjoint" type="fixed">
 		<parent link="l_ankle"/>
@@ -134,5 +244,16 @@
 		<axis xyz="0 0 0"/>
 	</joint>
-	<link name="LFsrRearCenter_frame"/>
+	<link name="LFsrRearCenter_frame">
+		<collision>
+			<geometry>
+				<box size="0.01 0.01 0.005"/>
+			</geometry>
+			<origin rpy="0 0 0" xyz="0 0 0"/>
+		</collision>
+		<inertial>
+			<mass value="2e-06"/>
+			<inertia ixx="1.1e-09" ixy="0" ixz="0" iyy="1.1e-09" iyz="0" izz="1.1e-09"/>
+		</inertial>
+	</link>
 	<joint name="LFoot/FSR/CenterRear_sensor_fixedjoint" type="fixed">
 		<parent link="l_ankle"/>
@@ -154,5 +275,16 @@
 		<origin rpy="-1.57079632679 0 -1.57079632679" xyz="0 0 0"/>
 	</joint>
-	<link name="LFsrFToeFrontRight_frame"/>
+	<link name="LFsrFToeFrontRight_frame">
+		<collision>
+			<geometry>
+				<box size="0.01 0.01 0.005"/>
+			</geometry>
+			<origin rpy="0 0 0" xyz="0 0 0"/>
+		</collision>
+		<inertial>
+			<mass value="2e-06"/>
+			<inertia ixx="1.1e-09" ixy="0" ixz="0" iyy="1.1e-09" iyz="0" izz="1.1e-09"/>
+		</inertial>
+	</link>
 	<joint name="LFoot/FSR/ToeFrontRight_sensor_fixedjoint" type="fixed">
 		<parent link="l_ankle"/>
@@ -161,5 +293,16 @@
 		<axis xyz="0 0 0"/>
 	</joint>
-	<link name="RFsrHeelLeft_frame"/>
+	<link name="RFsrHeelLeft_frame">
+		<collision>
+			<geometry>
+				<box size="0.01 0.01 0.005"/>
+			</geometry>
+			<origin rpy="0 0 0" xyz="0 0 0"/>
+		</collision>
+		<inertial>
+			<mass value="2e-06"/>
+			<inertia ixx="1.1e-09" ixy="0" ixz="0" iyy="1.1e-09" iyz="0" izz="1.1e-09"/>
+		</inertial>
+	</link>
 	<joint name="RFoot/FSR/HeelLeft_sensor_fixedjoint" type="fixed">
 		<parent link="r_ankle"/>
@@ -175,5 +318,16 @@
 		<axis xyz="0 0 0"/>
 	</joint>
-	<link name="LFsrFrontCenter_frame"/>
+	<link name="LFsrFrontCenter_frame">
+		<collision>
+			<geometry>
+				<box size="0.01 0.01 0.005"/>
+			</geometry>
+			<origin rpy="0 0 0" xyz="0 0 0"/>
+		</collision>
+		<inertial>
+			<mass value="2e-06"/>
+			<inertia ixx="1.1e-09" ixy="0" ixz="0" iyy="1.1e-09" iyz="0" izz="1.1e-09"/>
+		</inertial>
+	</link>
 	<joint name="LFoot/FSR/CenterFront_sensor_fixedjoint" type="fixed">
 		<parent link="l_ankle"/>
@@ -182,5 +336,16 @@
 		<axis xyz="0 0 0"/>
 	</joint>
-	<link name="RFsrFToeFrontLeft_frame"/>
+	<link name="RFsrFToeFrontLeft_frame">
+		<collision>
+			<geometry>
+				<box size="0.01 0.01 0.005"/>
+			</geometry>
+			<origin rpy="0 0 0" xyz="0 0 0"/>
+		</collision>
+		<inertial>
+			<mass value="2e-06"/>
+			<inertia ixx="1.1e-09" ixy="0" ixz="0" iyy="1.1e-09" iyz="0" izz="1.1e-09"/>
+		</inertial>
+	</link>
 	<joint name="RFoot/FSR/ToeFrontLeft_sensor_fixedjoint" type="fixed">
 		<parent link="r_ankle"/>
@@ -189,5 +354,16 @@
 		<axis xyz="0 0 0"/>
 	</joint>
-	<link name="LFsrFToeFrontLeft_frame"/>
+	<link name="LFsrFToeFrontLeft_frame">
+		<collision>
+			<geometry>
+				<box size="0.01 0.01 0.005"/>
+			</geometry>
+			<origin rpy="0 0 0" xyz="0 0 0"/>
+		</collision>
+		<inertial>
+			<mass value="2e-06"/>
+			<inertia ixx="1.1e-09" ixy="0" ixz="0" iyy="1.1e-09" iyz="0" izz="1.1e-09"/>
+		</inertial>
+	</link>
 	<joint name="LFoot/FSR/ToeFrontLeft_sensor_fixedjoint" type="fixed">
 		<parent link="l_ankle"/>
