Commit message: regenerated URDF

File: romeo_description/urdf/romeo_generated_urdf/romeo.urdf (robot description, URDF)
Before this commit: robot RomeoH37, 96 links, 95 joints
Links:
- added link CameraDepth_optical_frame
Joints:
- added joint CameraDepth_optical_frame_fixedjoint: type fixed, parent CameraDepth_frame, child CameraDepth_optical_frame, origin xyz=0 0 0 rpy=2.0043951 0 1.57079632679
- joint CameraDepth_joint: origin xyz=0.1403 -0.04708 0.14655 rpy=2.0043951 0 1.57079632679 -> xyz=0.1403 -0.04708 0.14655 rpy=0 0 0
